File: sepic2.kicad_sch (KiCad schematic)
At the start: 8 parts, among them Q1 T2N7002BK

Commit message: fix part number
Parts:
- Q1: Mouser part no. 757-T2N7002BKLM -> 757-T2N7002BKLM
Changed lines of the file:
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@@
 			)
 		)
-		(property "Mouser part no." " 757-T2N7002BKLM "
+		(property "Mouser part no." " 757-T2N7002BKLM"
 			(at 106.68 69.85 0)
 			(effects
