File: shifter.kicad_sch (KiCad schematic)
At the start: 19 parts, among them Q4 BC547, Q7 BC547, Q8 BC547, Q9 BC547

Commit message: change resistor part numbers to right sized ones
Parts:
- R14, R16, R17, R18: Mouser part no. 603-MFR-25FTE52-27K -> 603-MFR-12FTF52-27K
Changed lines of the file:
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@@
 			)
 		)
-		(property "Mouser part no." " 603-MFR-25FTE52-27K"
+		(property "Mouser part no." " 603-MFR-12FTF52-27K"
 			(at 92.71 121.92 0)
 			(effects
@@
 			)
 		)
-		(property "Mouser part no." " 603-MFR-25FTE52-27K"
+		(property "Mouser part no." " 603-MFR-12FTF52-27K"
 			(at 92.71 146.05 0)
 			(effects
@@
 			)
 		)
-		(property "Mouser part no." " 603-MFR-25FTE52-27K"
+		(property "Mouser part no." " 603-MFR-12FTF52-27K"
 			(at 92.71 97.79 0)
 			(effects
@@
 			)
 		)
-		(property "Mouser part no." " 603-MFR-25FTE52-27K"
+		(property "Mouser part no." " 603-MFR-12FTF52-27K"
 			(at 92.71 73.66 0)
 			(effects

Commit message: change to cute little (cheaper) SMD diodes
Parts:
- D10, D11, D12, D2, D3, D4, D5, D6, D7, D8, D9: value 1N4004 -> FDLL4148; footprint Diode_THT:D_DO-41_SOD81_P10.16mm_Horizontal -> Diode_SMD:D_1206_3216Metric_Pad1.42x1.75mm_HandSolder; Mouser part no. 637-1N4004GP -> 512-FDLL4148
Changed lines of the file:
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@@
 			)
 		)
-		(property "Value" "1N4004"
+		(property "Value" "FDLL4148"
 			(at 158.75 173.99 0)
 			(effects
@@
 			)
 		)
-		(property "Footprint" "Diode_THT:D_DO-41_SOD81_P10.16mm_Horizontal"
+		(property "Footprint" "Diode_SMD:D_1206_3216Metric_Pad1.42x1.75mm_HandSolder"
 			(at 158.75 173.355 0)
 			(effects
@@
 			)
 		)
-		(property "Datasheet" "http://www.vishay.com/docs/88503/1n4001.pdf"
+		(property "Datasheet" "https://au.mouser.com/datasheet/2/308/1N914_D-2309448.pdf"
 			(at 158.75 177.8 0)
 			(effects
@@
 			)
 		)
-		(property "Mouser part no." " 637-1N4004GP "
+		(property "Mouser part no." " 512-FDLL4148"
 			(at 158.75 177.8 0)
 			(effects
@@
 			)
 		)
-		(property "Value" "1N4004"
+		(property "Value" "FDLL4148"
 			(at 158.75 123.19 0)
 			(effects
@@
 			)
 		)
-		(property "Footprint" "Diode_THT:D_DO-41_SOD81_P10.16mm_Horizontal"
+		(property "Footprint" "Diode_SMD:D_1206_3216Metric_Pad1.42x1.75mm_HandSolder"
 			(at 158.75 122.555 0)
 			(effects
@@
 			)
 		)
-		(property "Datasheet" "http://www.vishay.com/docs/88503/1n4001.pdf"
+		(property "Datasheet" "https://au.mouser.com/datasheet/2/308/1N914_D-2309448.pdf"
 			(at 158.75 127 0)
 			(effects
@@
 			)
 		)
-		(property "Mouser part no." " 637-1N4004GP "
+		(property "Mouser part no." " 512-FDLL4148"
 			(at 158.75 127 0)
 			(effects
@@
 			)
 		)
-		(property "Value" "1N4004"
+		(property "Value" "FDLL4148"
 			(at 158.75 59.69 0)
 			(effects
@@
 			)
 		)
-		(property "Footprint" "Diode_THT:D_DO-41_SOD81_P10.16mm_Horizontal"
+		(property "Footprint" "Diode_SMD:D_1206_3216Metric_Pad1.42x1.75mm_HandSolder"
 			(at 158.75 59.055 0)
 			(effects
@@
 			)
 		)
-		(property "Datasheet" "http://www.vishay.com/docs/88503/1n4001.pdf"
+		(property "Datasheet" "https://au.mouser.com/datasheet/2/308/1N914_D-2309448.pdf"
 			(at 158.75 63.5 0)
 			(effects
@@
 			)
 		)
-		(property "Mouser part no." " 637-1N4004GP "
+		(property "Mouser part no." " 512-FDLL4148"
 			(at 158.75 63.5 0)
 			(effects
@@
 			)
 		)
-		(property "Value" "1N4004"
+		(property "Value" "FDLL4148"
 			(at 158.75 72.39 0)
 			(effects
@@
 			)
 		)
-		(property "Footprint" "Diode_THT:D_DO-41_SOD81_P10.16mm_Horizontal"
+		(property "Footprint" "Diode_SMD:D_1206_3216Metric_Pad1.42x1.75mm_HandSolder"
 			(at 158.75 71.755 0)
 			(effects
@@
 			)
 		)
-		(property "Datasheet" "http://www.vishay.com/docs/88503/1n4001.pdf"
+		(property "Datasheet" "https://au.mouser.com/datasheet/2/308/1N914_D-2309448.pdf"
 			(at 158.75 76.2 0)
 			(effects
@@
 			)
 		)
-		(property "Mouser part no." " 637-1N4004GP "
+		(property "Mouser part no." " 512-FDLL4148"
 			(at 158.75 76.2 0)
 			(effects
@@
 			)
 		)
-		(property "Value" "1N4004"
+		(property "Value" "FDLL4148"
 			(at 158.75 161.29 0)
 			(effects
@@
 			)
 		)
-		(property "Footprint" "Diode_THT:D_DO-41_SOD81_P10.16mm_Horizontal"
+		(property "Footprint" "Diode_SMD:D_1206_3216Metric_Pad1.42x1.75mm_HandSolder"
 			(at 158.75 160.655 0)
 			(effects
@@
 			)
 		)
-		(property "Datasheet" "http://www.vishay.com/docs/88503/1n4001.pdf"
+		(property "Datasheet" "https://au.mouser.com/datasheet/2/308/1N914_D-2309448.pdf"
 			(at 158.75 165.1 0)
 			(effects
@@
 			)
 		)
-		(property "Mouser part no." " 637-1N4004GP "
+		(property "Mouser part no." " 512-FDLL4148"
 			(at 158.75 165.1 0)
 			(effects
@@
 			)
 		)
-		(property "Value" "1N4004"
+		(property "Value" "FDLL4148"
 			(at 158.75 110.49 0)
 			(effects
@@
 			)
 		)
-		(property "Footprint" "Diode_THT:D_DO-41_SOD81_P10.16mm_Horizontal"
+		(property "Footprint" "Diode_SMD:D_1206_3216Metric_Pad1.42x1.75mm_HandSolder"
 			(at 158.75 109.855 0)
 			(effects
@@
 			)
 		)
-		(property "Datasheet" "http://www.vishay.com/docs/88503/1n4001.pdf"
+		(property "Datasheet" "https://au.mouser.com/datasheet/2/308/1N914_D-2309448.pdf"
 			(at 158.75 114.3 0)
 			(effects
@@
 			)
 		)
-		(property "Mouser part no." " 637-1N4004GP "
+		(property "Mouser part no." " 512-FDLL4148"
 			(at 158.75 114.3 0)
 			(effects
@@
 			)
 		)
-		(property "Value" "1N4004"
+		(property "Value" "FDLL4148"
 			(at 158.75 85.09 0)
 			(effects
@@
 			)
 		)
-		(property "Footprint" "Diode_THT:D_DO-41_SOD81_P10.16mm_Horizontal"
+		(property "Footprint" "Diode_SMD:D_1206_3216Metric_Pad1.42x1.75mm_HandSolder"
 			(at 158.75 84.455 0)
 			(effects
@@
 			)
 		)
-		(property "Datasheet" "http://www.vishay.com/docs/88503/1n4001.pdf"
+		(property "Datasheet" "https://au.mouser.com/datasheet/2/308/1N914_D-2309448.pdf"
 			(at 158.75 88.9 0)
 			(effects
@@
 			)
 		)
-		(property "Mouser part no." " 637-1N4004GP "
+		(property "Mouser part no." " 512-FDLL4148"
 			(at 158.75 88.9 0)
 			(effects
@@
 			)
 		)
-		(property "Value" "1N4004"
+		(property "Value" "FDLL4148"
 			(at 158.75 148.59 0)
 			(effects
@@
 			)
 		)
-		(property "Footprint" "Diode_THT:D_DO-41_SOD81_P10.16mm_Horizontal"
+		(property "Footprint" "Diode_SMD:D_1206_3216Metric_Pad1.42x1.75mm_HandSolder"
 			(at 158.75 147.955 0)
 			(effects
@@
 			)
 		)
-		(property "Datasheet" "http://www.vishay.com/docs/88503/1n4001.pdf"
+		(property "Datasheet" "https://au.mouser.com/datasheet/2/308/1N914_D-2309448.pdf"
 			(at 158.75 152.4 0)
 			(effects
@@
 			)
 		)
-		(property "Mouser part no." " 637-1N4004GP "
+		(property "Mouser part no." " 512-FDLL4148"
 			(at 158.75 152.4 0)
 			(effects
@@
 			)
 		)
-		(property "Value" "1N4004"
+		(property "Value" "FDLL4148"
 			(at 158.75 46.99 0)
 			(effects
@@
 			)
 		)
-		(property "Footprint" "Diode_THT:D_DO-41_SOD81_P10.16mm_Horizontal"
+		(property "Footprint" "Diode_SMD:D_1206_3216Metric_Pad1.42x1.75mm_HandSolder"
 			(at 158.75 46.355 0)
 			(effects
@@
 			)
 		)
-		(property "Datasheet" "http://www.vishay.com/docs/88503/1n4001.pdf"
+		(property "Datasheet" "https://au.mouser.com/datasheet/2/308/1N914_D-2309448.pdf"
 			(at 158.75 50.8 0)
 			(effects
@@
 			)
 		)
-		(property "Mouser part no." " 637-1N4004GP "
+		(property "Mouser part no." " 512-FDLL4148"
 			(at 158.75 50.8 0)
 			(effects
@@
 			)
 		)
-		(property "Value" "1N4004"
+		(property "Value" "FDLL4148"
 			(at 158.75 97.79 0)
 			(effects
@@
 			)
 		)
-		(property "Footprint" "Diode_THT:D_DO-41_SOD81_P10.16mm_Horizontal"
+		(property "Footprint" "Diode_SMD:D_1206_3216Metric_Pad1.42x1.75mm_HandSolder"
 			(at 158.75 97.155 0)
 			(effects
@@
 			)
 		)
-		(property "Datasheet" "http://www.vishay.com/docs/88503/1n4001.pdf"
+		(property "Datasheet" "https://au.mouser.com/datasheet/2/308/1N914_D-2309448.pdf"
 			(at 158.75 101.6 0)
 			(effects
@@
 			)
 		)
-		(property "Mouser part no." " 637-1N4004GP "
+		(property "Mouser part no." " 512-FDLL4148"
 			(at 158.75 101.6 0)
 			(effects
@@
 			)
 		)
-		(property "Value" "1N4004"
+		(property "Value" "FDLL4148"
 			(at 158.75 135.89 0)
 			(effects
@@
 			)
 		)
-		(property "Footprint" "Diode_THT:D_DO-41_SOD81_P10.16mm_Horizontal"
+		(property "Footprint" "Diode_SMD:D_1206_3216Metric_Pad1.42x1.75mm_HandSolder"
 			(at 158.75 135.255 0)
 			(effects
@@
 			)
 		)
-		(property "Datasheet" "http://www.vishay.com/docs/88503/1n4001.pdf"
+		(property "Datasheet" "https://au.mouser.com/datasheet/2/308/1N914_D-2309448.pdf"
 			(at 158.75 139.7 0)
 			(effects
@@
 			)
 		)
-		(property "Mouser part no." " 637-1N4004GP "
+		(property "Mouser part no." " 512-FDLL4148"
 			(at 158.75 139.7 0)
 			(effects

Commit message: change most NPNs to SMD ones
Parts:
- Q4, Q7, Q8, Q9: value BC547 -> BC847C; footprint Package_TO_SOT_THT:TO-92_Inline -> Package_TO_SOT_SMD:SOT-23_Handsoldering; Mouser part no. 637-BC547CBK -> 771-BC847C-T/R
Changed lines of the file:
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@@
 			)
 		)
-		(property "Value" "BC547"
+		(property "Value" "BC847C"
 			(at 109.22 147.3199 0)
 			(effects
@@
 			)
 		)
-		(property "Footprint" "Package_TO_SOT_THT:TO-92_Inline"
+		(property "Footprint" "Package_TO_SOT_SMD:SOT-23_Handsoldering"
 			(at 109.22 147.955 0)
 			(effects
@@
 			)
 		)
-		(property "Datasheet" "https://www.onsemi.com/pub/Collateral/BC550-D.pdf"
+		(property "Datasheet" "https://au.mouser.com/datasheet/2/916/BC847X_SER-3081381.pdf"
 			(at 104.14 146.05 0)
 			(effects
@@
 			)
 		)
-		(property "Mouser part no." " 637-BC547CBK"
+		(property "Mouser part no." " 771-BC847C-T/R"
 			(at 104.14 146.05 0)
 			(effects
@@
 			)
 		)
-		(property "Value" "BC547"
+		(property "Value" "BC847C"
 			(at 109.22 74.9299 0)
 			(effects
@@
 			)
 		)
-		(property "Footprint" "Package_TO_SOT_THT:TO-92_Inline"
+		(property "Footprint" "Package_TO_SOT_SMD:SOT-23_Handsoldering"
 			(at 109.22 75.565 0)
 			(effects
@@
 			)
 		)
-		(property "Datasheet" "https://www.onsemi.com/pub/Collateral/BC550-D.pdf"
+		(property "Datasheet" "https://au.mouser.com/datasheet/2/916/BC847X_SER-3081381.pdf"
 			(at 104.14 73.66 0)
 			(effects
@@
 			)
 		)
-		(property "Mouser part no." " 637-BC547CBK"
+		(property "Mouser part no." " 771-BC847C-T/R"
 			(at 104.14 73.66 0)
 			(effects
@@
 			)
 		)
-		(property "Value" "BC547"
+		(property "Value" "BC847C"
 			(at 109.22 123.1899 0)
 			(effects
@@
 			)
 		)
-		(property "Footprint" "Package_TO_SOT_THT:TO-92_Inline"
+		(property "Footprint" "Package_TO_SOT_SMD:SOT-23_Handsoldering"
 			(at 109.22 123.825 0)
 			(effects
@@
 			)
 		)
-		(property "Datasheet" "https://www.onsemi.com/pub/Collateral/BC550-D.pdf"
+		(property "Datasheet" "https://au.mouser.com/datasheet/2/916/BC847X_SER-3081381.pdf"
 			(at 104.14 121.92 0)
 			(effects
@@
 			)
 		)
-		(property "Mouser part no." " 637-BC547CBK"
+		(property "Mouser part no." " 771-BC847C-T/R"
 			(at 104.14 121.92 0)
 			(effects
@@
 			)
 		)
-		(property "Value" "BC547"
+		(property "Value" "BC847C"
 			(at 109.22 99.0599 0)
 			(effects
@@
 			)
 		)
-		(property "Footprint" "Package_TO_SOT_THT:TO-92_Inline"
+		(property "Footprint" "Package_TO_SOT_SMD:SOT-23_Handsoldering"
 			(at 109.22 99.695 0)
 			(effects
@@
 			)
 		)
-		(property "Datasheet" "https://www.onsemi.com/pub/Collateral/BC550-D.pdf"
+		(property "Datasheet" "https://au.mouser.com/datasheet/2/916/BC847X_SER-3081381.pdf"
 			(at 104.14 97.79 0)
 			(effects
@@
 			)
 		)
-		(property "Mouser part no." " 637-BC547CBK"
+		(property "Mouser part no." " 771-BC847C-T/R"
 			(at 104.14 97.79 0)
 			(effects

Commit message: change some resistors to SMD
Parts:
- R14, R16, R17, R18: footprint Resistor_THT:R_Axial_DIN0204_L3.6mm_D1.6mm_P7.62mm_Horizontal -> Resistor_SMD:R_0805_2012Metric_Pad1.20x1.40mm_HandSolder; Mouser part no. 603-MFR-12FTF52-27K -> 603-RE0805FRE0727KL
Changed lines of the file:
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@@
 			)
 		)
-		(property "Footprint" "Resistor_THT:R_Axial_DIN0204_L3.6mm_D1.6mm_P7.62mm_Horizontal"
+		(property "Footprint" "Resistor_SMD:R_0805_2012Metric_Pad1.20x1.40mm_HandSolder"
 			(at 92.71 123.698 90)
 			(effects
@@
 			)
 		)
-		(property "Mouser part no." " 603-MFR-12FTF52-27K"
+		(property "Mouser part no." " 603-RE0805FRE0727KL"
 			(at 92.71 121.92 0)
 			(effects
@@
 			)
 		)
-		(property "Footprint" "Resistor_THT:R_Axial_DIN0204_L3.6mm_D1.6mm_P7.62mm_Horizontal"
+		(property "Footprint" "Resistor_SMD:R_0805_2012Metric_Pad1.20x1.40mm_HandSolder"
 			(at 92.71 147.828 90)
 			(effects
@@
 			)
 		)
-		(property "Mouser part no." " 603-MFR-12FTF52-27K"
+		(property "Mouser part no." " 603-RE0805FRE0727KL"
 			(at 92.71 146.05 0)
 			(effects
@@
 			)
 		)
-		(property "Footprint" "Resistor_THT:R_Axial_DIN0204_L3.6mm_D1.6mm_P7.62mm_Horizontal"
+		(property "Footprint" "Resistor_SMD:R_0805_2012Metric_Pad1.20x1.40mm_HandSolder"
 			(at 92.71 99.568 90)
 			(effects
@@
 			)
 		)
-		(property "Mouser part no." " 603-MFR-12FTF52-27K"
+		(property "Mouser part no." " 603-RE0805FRE0727KL"
 			(at 92.71 97.79 0)
 			(effects
@@
 			)
 		)
-		(property "Footprint" "Resistor_THT:R_Axial_DIN0204_L3.6mm_D1.6mm_P7.62mm_Horizontal"
+		(property "Footprint" "Resistor_SMD:R_0805_2012Metric_Pad1.20x1.40mm_HandSolder"
 			(at 92.71 75.438 90)
 			(effects
@@
 			)
 		)
-		(property "Mouser part no." " 603-MFR-12FTF52-27K"
+		(property "Mouser part no." " 603-RE0805FRE0727KL"
 			(at 92.71 73.66 0)
 			(effects

Commit message: fix clock signal level shifting
Parts:
- added R19: 27k, Resistor_SMD:R_0805_2012Metric_Pad1.20x1.40mm_HandSolder, symbol Device:R
Connections:
- net ~{4MHz} CMOS: now also R19.2
- new net +3V3: R19.1
Changed lines of the file:
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@@
 	(generator_version "8.0")
 	(paper "A4")
+	(junction
+		(at 152.4 101.6)
+		(diameter 0)
+		(color 0 0 0 0)
+	)
 	(wire
 		(pts
@@
 	(wire
 		(pts
+			(xy 149.86 99.06) (xy 152.4 99.06)
+		)
+		(stroke
+			(width 0)
+			(type default)
+		)
+	)
+	(wire
+		(pts
 			(xy 162.56 114.3) (xy 165.1 114.3)
 		)
@@
 	(wire
 		(pts
+			(xy 139.7 101.6) (xy 152.4 101.6)
+		)
+		(stroke
+			(width 0)
+			(type default)
+		)
+	)
+	(wire
+		(pts
+			(xy 106.68 138.43) (xy 109.22 138.43)
+		)
+		(stroke
+			(width 0)
+			(type default)
+		)
+	)
+	(wire
+		(pts
+			(xy 152.4 50.8) (xy 154.94 50.8)
+		)
+		(stroke
+			(width 0)
+			(type default)
+		)
+	)
+	(wire
+		(pts
+			(xy 162.56 63.5) (xy 165.1 63.5)
+		)
+		(stroke
+			(width 0)
+			(type default)
+		)
+	)
+	(wire
+		(pts
+			(xy 96.52 97.79) (xy 99.06 97.79)
+		)
+		(stroke
+			(width 0)
+			(type default)
+		)
+	)
+	(wire
+		(pts
+			(xy 106.68 90.17) (xy 109.22 90.17)
+		)
+		(stroke
+			(width 0)
+			(type default)
+		)
+	)
+	(wire
+		(pts
+			(xy 152.4 114.3) (xy 154.94 114.3)
+		)
+		(stroke
+			(width 0)
+			(type default)
+		)
+	)
+	(wire
+		(pts
+			(xy 162.56 152.4) (xy 165.1 152.4)
+		)
+		(stroke
+			(width 0)
+			(type default)
+		)
+	)
+	(wire
+		(pts
+			(xy 152.4 99.06) (xy 152.4 101.6)
+		)
+		(stroke
+			(width 0)
+			(type default)
+		)
+	)
+	(wire
+		(pts
+			(xy 106.68 116.84) (xy 106.68 114.3)
+		)
+		(stroke
+			(width 0)
+			(type default)
+		)
+	)
+	(wire
+		(pts
+			(xy 152.4 63.5) (xy 154.94 63.5)
+		)
+		(stroke
+			(width 0)
+			(type default)
+		)
+	)
+	(wire
+		(pts
+			(xy 162.56 76.2) (xy 165.1 76.2)
+		)
+		(stroke
+			(width 0)
+			(type default)
+		)
+	)
+	(wire
+		(pts
+			(xy 152.4 152.4) (xy 154.94 152.4)
+		)
+		(stroke
+			(width 0)
+			(type default)
+		)
+	)
+	(wire
+		(pts
+			(xy 162.56 50.8) (xy 165.1 50.8)
+		)
+		(stroke
+			(width 0)
+			(type default)
+		)
+	)
+	(wire
+		(pts
+			(xy 106.68 78.74) (xy 106.68 81.28)
+		)
+		(stroke
+			(width 0)
+			(type default)
+		)
+	)
+	(wire
+		(pts
 			(xy 152.4 101.6) (xy 154.94 101.6)
 		)
@@
 	(wire
 		(pts
-			(xy 106.68 138.43) (xy 109.22 138.43)
-		)
-		(stroke
-			(width 0)
-			(type default)
-		)
-	)
-	(wire
-		(pts
-			(xy 152.4 50.8) (xy 154.94 50.8)
-		)
-		(stroke
-			(width 0)
-			(type default)
-		)
-	)
-	(wire
-		(pts
-			(xy 162.56 63.5) (xy 165.1 63.5)
-		)
-		(stroke
-			(width 0)
-			(type default)
-		)
-	)
-	(wire
-		(pts
-			(xy 96.52 97.79) (xy 99.06 97.79)
-		)
-		(stroke
-			(width 0)
-			(type default)
-		)
-	)
-	(wire
-		(pts
-			(xy 106.68 90.17) (xy 109.22 90.17)
-		)
-		(stroke
-			(width 0)
-			(type default)
-		)
-	)
-	(wire
-		(pts
-			(xy 152.4 114.3) (xy 154.94 114.3)
-		)
-		(stroke
-			(width 0)
-			(type default)
-		)
-	)
-	(wire
-		(pts
-			(xy 162.56 152.4) (xy 165.1 152.4)
-		)
-		(stroke
-			(width 0)
-			(type default)
-		)
-	)
-	(wire
-		(pts
-			(xy 106.68 116.84) (xy 106.68 114.3)
-		)
-		(stroke
-			(width 0)
-			(type default)
-		)
-	)
-	(wire
-		(pts
-			(xy 152.4 63.5) (xy 154.94 63.5)
-		)
-		(stroke
-			(width 0)
-			(type default)
-		)
-	)
-	(wire
-		(pts
-			(xy 162.56 76.2) (xy 165.1 76.2)
-		)
-		(stroke
-			(width 0)
-			(type default)
-		)
-	)
-	(wire
-		(pts
-			(xy 152.4 152.4) (xy 154.94 152.4)
-		)
-		(stroke
-			(width 0)
-			(type default)
-		)
-	)
-	(wire
-		(pts
-			(xy 162.56 50.8) (xy 165.1 50.8)
-		)
-		(stroke
-			(width 0)
-			(type default)
-		)
-	)
-	(wire
-		(pts
-			(xy 106.68 78.74) (xy 106.68 81.28)
-		)
-		(stroke
-			(width 0)
-			(type default)
-		)
-	)
-	(wire
-		(pts
 			(xy 106.68 66.04) (xy 109.22 66.04)
 		)
@@
 	(wire
 		(pts
+			(xy 139.7 96.52) (xy 139.7 99.06)
+		)
+		(stroke
+			(width 0)
+			(type default)
+		)
+	)
+	(wire
+		(pts
 			(xy 162.56 88.9) (xy 165.1 88.9)
+		)
+		(stroke
+			(width 0)
+			(type default)
+		)
+	)
+	(wire
+		(pts
+			(xy 139.7 99.06) (xy 142.24 99.06)
 		)
 		(stroke
@@
 	(hierarchical_label "~{4MHz} CMOS"
 		(shape output)
-		(at 152.4 101.6 180)
+		(at 139.7 101.6 180)
 		(fields_autoplaced yes)
 		(effects
@@
 			)
 			(justify right)
+		)
+	)
+	(symbol
+		(lib_id "Device:R")
+		(at 146.05 99.06 90)
+		(unit 1)
+		(exclude_from_sim no)
+		(in_bom yes)
+		(on_board yes)
+		(dnp no)
+		(fields_autoplaced yes)
+		(property "Reference" "R19"
+			(at 146.05 92.71 90)
+			(effects
+				(font
+					(size 1.27 1.27)
+				)
+			)
+		)
+		(property "Value" "27k"
+			(at 146.05 95.25 90)
+			(effects
+				(font
+					(size 1.27 1.27)
+				)
+			)
+		)
+		(property "Footprint" "Resistor_SMD:R_0805_2012Metric_Pad1.20x1.40mm_HandSolder"
+			(at 146.05 100.838 90)
+			(effects
+				(font
+					(size 1.27 1.27)
+				)
+				(hide yes)
+			)
+		)
+		(property "Datasheet" "~"
+			(at 146.05 99.06 0)
+			(effects
+				(font
+					(size 1.27 1.27)
+				)
+				(hide yes)
+			)
+		)
+		(property "Description" "Resistor"
+			(at 146.05 99.06 0)
+			(effects
+				(font
+					(size 1.27 1.27)
+				)
+				(hide yes)
+			)
+		)
+		(property "Mouser part no." " 603-RE0805FRE0727KL"
+			(at 146.05 99.06 0)
+			(effects
+				(font
+					(size 1.27 1.27)
+				)
+				(hide yes)
+			)
+		)
+		(pin "2"
+		)
+		(pin "1"
+		)
+		(instances
+			(project "osborne-floppy-emulator"
+				(path "/a407fcbc-6d86-4aa2-968f-b2fcdecb9640/c000f981-768b-40ae-b27c-6b54380ce47a"
+					(reference "R19")
+					(unit 1)
+				)
+			)
 		)
 	)
@@
 					(unit 1)
 				)
+			)
+		)
+	)
+	(symbol
+		(lib_id "power:+3V3")
+		(at 139.7 96.52 0)
+		(unit 1)
+		(exclude_from_sim no)
+		(in_bom yes)
+		(on_board yes)
+		(dnp no)
+		(fields_autoplaced yes)
+		(property "Reference" "#PWR031"
+			(at 139.7 100.33 0)
+			(effects
+				(font
+					(size 1.27 1.27)
+				)
+				(hide yes)
+			)
+		)
+		(property "Value" "+3V3"
+			(at 139.7 91.44 0)
+			(effects
+				(font
+					(size 1.27 1.27)
+				)
+			)
+		)
+		(property "Footprint" ""
+			(at 139.7 96.52 0)
+			(effects
+				(font
+					(size 1.27 1.27)
+				)
+				(hide yes)
+			)
+		)
+		(property "Datasheet" ""
+			(at 139.7 96.52 0)
+			(effects
+				(font
+					(size 1.27 1.27)
+				)
+				(hide yes)
+			)
+		)
+		(property "Description" "Power symbol creates a global label with name \"+3V3\""
+			(at 139.7 96.52 0)
+			(effects
+				(font
+					(size 1.27 1.27)
+				)
+				(hide yes)
+			)
+		)
+		(pin "1"
+		)
+		(instances
+			(project "osborne-floppy-emulator"
+				(path "/a407fcbc-6d86-4aa2-968f-b2fcdecb9640/c000f981-768b-40ae-b27c-6b54380ce47a"
+					(reference "#PWR031")
+					(unit 1)
+				)
