File: connector.kicad_sch (KiCad schematic)
At the start: 4 parts, among them J1 Connector Out, J4 Connector In, Q5 BC547, Q6 BC547

Commit message: changed part numbers for connectors
Parts:
- J1: Mouser part no. 737-PH2-18-UA -> 649-67996-434HLF
- J4: Mouser part no. 737-RS2-20-G -> 710-61304021821
Changed lines of the file:
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@@
 			)
 		)
-		(property "Mouser part no." " 737-RS2-20-G"
+		(property "Mouser part no." " 710-61304021821"
 			(at 156.21 82.55 0)
 			(effects
@@
 			)
 		)
-		(property "Mouser part no." " 737-PH2-18-UA"
-			(at 156.21 134.62 0)
-			(effects
+		(property "Mouser part no." " 649-67996-434HLF"
+			(at 156.21 134.62 0)
+			(effects

Commit message: change pin headers to (more expensive) SMT ones
Parts:
- J1: footprint Connector_PinHeader_2.54mm:PinHeader_2x17_P2.54mm_Vertical -> Connector_PinHeader_2.54mm:PinHeader_2x17_P2.54mm_Vertical_SMD; Mouser part no. 649-67996-434HLF -> 855-M20-7812045
- J4: footprint Connector_PinSocket_2.54mm:PinSocket_2x17_P2.54mm_Vertical -> Connector_PinSocket_2.54mm:PinSocket_2x17_P2.54mm_Vertical_SMD
Changed lines of the file:
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@@
 			)
 		)
-		(property "Footprint" "Connector_PinSocket_2.54mm:PinSocket_2x17_P2.54mm_Vertical"
+		(property "Footprint" "Connector_PinSocket_2.54mm:PinSocket_2x17_P2.54mm_Vertical_SMD"
 			(at 156.21 82.55 0)
 			(effects
@@
 			)
 		)
-		(property "Footprint" "Connector_PinHeader_2.54mm:PinHeader_2x17_P2.54mm_Vertical"
+		(property "Footprint" "Connector_PinHeader_2.54mm:PinHeader_2x17_P2.54mm_Vertical_SMD"
 			(at 156.21 134.62 0)
 			(effects
@@
 			)
 		)
-		(property "Mouser part no." " 649-67996-434HLF"
+		(property "Mouser part no." " 855-M20-7812045"
 			(at 156.21 134.62 0)
 			(effects

Commit message: change most NPNs to SMD ones
Parts:
- Q5, Q6: value BC547 -> BC847C; footprint Package_TO_SOT_THT:TO-92_Inline -> Package_TO_SOT_SMD:SOT-23_Handsoldering; Mouser part no. 637-BC547CBK -> 771-BC847C-T/R
Changed lines of the file:
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@@
 			)
 		)
-		(property "Value" "BC547"
+		(property "Value" "BC847C"
 			(at 186.69 130.81 90)
 			(effects
@@
 			)
 		)
-		(property "Footprint" "Package_TO_SOT_THT:TO-92_Inline"
+		(property "Footprint" "Package_TO_SOT_SMD:SOT-23_Handsoldering"
 			(at 188.595 127 0)
 			(effects
@@
 			)
 		)
-		(property "Datasheet" "https://www.onsemi.com/pub/Collateral/BC550-D.pdf"
+		(property "Datasheet" "https://au.mouser.com/datasheet/2/916/BC847X_SER-3081381.pdf"
 			(at 186.69 121.92 0)
 			(effects
@@
 			)
 		)
-		(property "Mouser part no." " 637-BC547CBK"
+		(property "Mouser part no." " 771-BC847C-T/R"
 			(at 186.69 121.92 0)
 			(effects
@@
 			)
 		)
-		(property "Value" "BC547"
+		(property "Value" "BC847C"
 			(at 205.74 133.35 90)
 			(effects
@@
 			)
 		)
-		(property "Footprint" "Package_TO_SOT_THT:TO-92_Inline"
+		(property "Footprint" "Package_TO_SOT_SMD:SOT-23_Handsoldering"
 			(at 207.645 129.54 0)
 			(effects
@@
 			)
 		)
-		(property "Datasheet" "https://www.onsemi.com/pub/Collateral/BC550-D.pdf"
+		(property "Datasheet" "https://au.mouser.com/datasheet/2/916/BC847X_SER-3081381.pdf"
 			(at 205.74 124.46 0)
 			(effects
@@
 			)
 		)
-		(property "Mouser part no." " 637-BC547CBK"
+		(property "Mouser part no." " 771-BC847C-T/R"
 			(at 205.74 124.46 0)
 			(effects

Commit message: Change a whole bunch of stuff for v2
Connections:
- net FDD Enable renamed DS 1 Enable
- net DS 1 Enable: no longer Q6.2 (B)
- new net DS 2 Enable: Q6.2 (B)
Changed lines of the file:
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@@
-	)
-	(junction
-		(at 205.74 115.57)
-		(diameter 0)
-		(color 0 0 0 0)
 	)
 	(junction
@@
 	(wire
 		(pts
+			(xy 186.69 111.76) (xy 196.85 111.76)
+		)
+		(stroke
+			(width 0)
+			(type default)
+		)
+	)
+	(wire
+		(pts
 			(xy 143.51 144.78) (xy 143.51 142.24)
 		)
@@
 	(wire
 		(pts
-			(xy 186.69 115.57) (xy 186.69 116.84)
+			(xy 186.69 111.76) (xy 186.69 116.84)
 		)
 		(stroke
@@
 		(pts
 			(xy 163.83 134.62) (xy 168.91 134.62)
-		)
-		(stroke
-			(width 0)
-			(type default)
-		)
-	)
-	(wire
-		(pts
-			(xy 205.74 115.57) (xy 186.69 115.57)
 		)
 		(stroke
@@
 		)
 	)
+	(hierarchical_label "DS 1 Enable"
+		(shape input)
+		(at 196.85 111.76 0)
+		(fields_autoplaced yes)
+		(effects
+			(font
+				(size 1.27 1.27)
+			)
+			(justify left)
+		)
+	)
 	(hierarchical_label "~{Write Data}"
 		(shape output)
@@
 		)
 	)
-	(hierarchical_label "FDD Enable"
+	(hierarchical_label "DS 2 Enable"
 		(shape input)
 		(at 209.55 115.57 0)
