File: osborne-floppy-emulator.kicad_sch (KiCad schematic)
At the start: 2 parts, among them J2 USB_A, J3 SWD Connector

Commit message: Change a whole bunch of stuff for v2
Other:
- sheet Connector ports: added DS 1 Enable, DS 2 Enable; removed FDD Enable
- sheet Processor ports: added DS 1 Enable, DS 2 Enable; removed FDD Enable
Changed lines of the file:
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@@
+	(wire
+		(pts
+			(xy 104.14 172.72) (xy 161.29 172.72)
+		)
+		(stroke
+			(width 0)
+			(type default)
+		)
+	)
 	(wire
 		(pts
@@
 	(sheet
 		(at 161.29 104.14)
-		(size 29.21 68.58)
+		(size 29.21 72.39)
 		(fields_autoplaced yes)
 		(stroke
@@
 		)
 		(property "Sheetfile" "connector.kicad_sch"
-			(at 161.29 173.3046 0)
+			(at 161.29 177.1146 0)
 			(effects
 				(font
@@
 			)
 		)
-		(pin "FDD Enable" input
+		(pin "DS 1 Enable" input
 			(at 161.29 168.91 180)
+			(effects
+				(font
+					(size 1.27 1.27)
+				)
+				(justify left)
+			)
+		)
+		(pin "DS 2 Enable" input
+			(at 161.29 172.72 180)
 			(effects
 				(font
@@
 	(sheet
 		(at 81.28 104.14)
-		(size 22.86 68.58)
+		(size 22.86 72.39)
 		(fields_autoplaced yes)
 		(stroke
@@
 		)
 		(property "Sheetfile" "rp2040.kicad_sch"
-			(at 81.28 173.3046 0)
+			(at 81.28 177.1146 0)
 			(effects
 				(font
@@
 			)
 		)
-		(pin "FDD Enable" output
-			(at 104.14 168.91 0)
-			(effects
-				(font
-					(size 1.27 1.27)
-				)
-				(justify right)
-			)
-		)
 		(pin "~{TG43}" input
 			(at 104.14 107.95 0)
@@
 			(effects
 				(font
+					(size 1.27 1.27)
+				)
+				(justify right)
+			)
+		)
+		(pin "DS 2 Enable" output
+			(at 104.14 172.72 0)
+			(effects
+				(font
+					(size 1.27 1.27)
+				)
+				(justify right)
+			)
+		)
+		(pin "DS 1 Enable" output
+			(at 104.14 168.91 0)
+			(effects
+				(font
