File: regulator.kicad_sch (KiCad schematic)
At the start: 17 parts, among them Q1 BC557, Q2 BC547, U3 TL494

Commit message: change resistor part numbers to right sized ones
Parts:
- R10: Mouser part no. 603-MFR-25FTE52-12K -> 603-MFR-12FTF52-12K
- R12, R13, R2, R3, R5: Mouser part no. 603-MFR-25FTE52-27K -> 603-MFR-12FTF52-27K
- R4: Mouser part no. 603-MFR-25FTE52-3K6 -> 603-MFR-12FTF52-3K6
- R6: Mouser part no. 603-MFR-25FTE52-7K5 -> 603-MFR-12FTF52-7K5
- R9: Mouser part no. 603-MFR-25FTE52-56R -> 603-MFR-12FTF52-56R
Changed lines of the file:
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@@
 			)
 		)
-		(property "Mouser part no." " 603-MFR-25FTE52-27K"
+		(property "Mouser part no." " 603-MFR-12FTF52-27K"
 			(at 118.11 97.79 0)
 			(effects
@@
 			)
 		)
-		(property "Mouser part no." " 603-MFR-25FTE52-3K6 "
+		(property "Mouser part no." " 603-MFR-12FTF52-3K6 "
 			(at 144.78 104.14 0)
 			(effects
@@
 			)
 		)
-		(property "Mouser part no." " 603-MFR-25FTE52-27K"
+		(property "Mouser part no." " 603-MFR-12FTF52-27K"
 			(at 187.96 102.87 0)
 			(effects
@@
 			)
 		)
-		(property "Mouser part no." " 603-MFR-25FTE52-56R"
+		(property "Mouser part no." " 603-MFR-12FTF52-56R"
 			(at 102.87 93.98 0)
 			(effects
@@
 			)
 		)
-		(property "Mouser part no." " 603-MFR-25FTE52-27K"
+		(property "Mouser part no." " 603-MFR-12FTF52-27K"
 			(at 151.13 85.09 0)
 			(effects
@@
 			)
 		)
-		(property "Mouser part no." " 603-MFR-25FTE52-27K"
+		(property "Mouser part no." " 603-MFR-12FTF52-27K"
 			(at 194.31 92.71 0)
 			(effects
@@
 			)
 		)
-		(property "Mouser part no." " 603-MFR-25FTE52-27K"
+		(property "Mouser part no." " 603-MFR-12FTF52-27K"
 			(at 107.95 99.06 0)
 			(effects
@@
 			)
 		)
-		(property "Mouser part no." " 603-MFR-25FTE52-7K5"
+		(property "Mouser part no." " 603-MFR-12FTF52-7K5"
 			(at 118.11 109.22 0)
 			(effects
@@
 			)
 		)
-		(property "Mouser part no." " 603-MFR-25FTE52-12K"
+		(property "Mouser part no." " 603-MFR-12FTF52-12K"
 			(at 143.51 119.38 0)
 			(effects

Commit message: fixed issue with OCP comparator polarity
Connections:
- net GND: now also U3.16 (2IN+); no longer U3.15 (2IN-)
- net at R13.2, R9.1: now also U3.15 (2IN-); no longer U3.16 (2IN+)
Changed lines of the file:
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@@
-	(wire
-		(pts
-			(xy 154.94 96.52) (xy 146.05 96.52)
-		)
-		(stroke
-			(width 0)
-			(type default)
-		)
-	)
 	(wire
 		(pts
@@
 	(wire
 		(pts
-			(xy 148.59 86.36) (xy 148.59 99.06)
+			(xy 148.59 86.36) (xy 148.59 96.52)
+		)
+		(stroke
+			(width 0)
+			(type default)
+		)
+	)
+	(wire
+		(pts
+			(xy 146.05 99.06) (xy 154.94 99.06)
 		)
 		(stroke
@@
 	(wire
 		(pts
-			(xy 148.59 99.06) (xy 154.94 99.06)
-		)
-		(stroke
-			(width 0)
-			(type default)
-		)
-	)
-	(wire
-		(pts
 			(xy 97.79 101.6) (xy 97.79 104.14)
 		)
@@
 	(wire
 		(pts
-			(xy 146.05 96.52) (xy 146.05 88.9)
-		)
-		(stroke
-			(width 0)
-			(type default)
-		)
-	)
-	(wire
-		(pts
 			(xy 153.67 123.19) (xy 153.67 124.46)
 		)
@@
 	(wire
 		(pts
+			(xy 146.05 88.9) (xy 146.05 99.06)
+		)
+		(stroke
+			(width 0)
+			(type default)
+		)
+	)
+	(wire
+		(pts
 			(xy 118.11 104.14) (xy 140.97 104.14)
 		)
@@
 		)
 		(stroke
+			(width 0)
+			(type default)
+		)
+	)
+	(wire
+		(pts
+			(xy 148.59 96.52) (xy 154.94 96.52)
+		)
+		(stroke

Commit message: changed regulator IC to TSSOP version
Parts:
- U3: footprint Package_DIP:DIP-16_W7.62mm_Socket -> Package_SO:TSSOP-16_4.4x5mm_P0.65mm; Mouser part no. 595-TL494CNE4 -> 595-TL494CPWR
Changed lines of the file:
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@@
 			)
 		)
-		(property "Footprint" "Package_DIP:DIP-16_W7.62mm_Socket"
+		(property "Footprint" "Package_SO:TSSOP-16_4.4x5mm_P0.65mm"
 			(at 167.64 104.14 0)
 			(effects
@@
 			)
 		)
-		(property "Mouser part no." " 595-TL494CNE4"
+		(property "Mouser part no." " 595-TL494CPWR"
 			(at 167.64 104.14 0)
 			(effects

Commit message: Change a whole bunch of stuff for v2
Parts:
- R13: footprint Resistor_THT:R_Axial_DIN0204_L3.6mm_D1.6mm_P7.62mm_Horizontal -> Resistor_SMD:R_0805_2012Metric_Pad1.20x1.40mm_HandSolder; Mouser part no. 603-MFR-12FTF52-27K -> 603-RE0805FRE0727KL
- R4: footprint Resistor_THT:R_Axial_DIN0204_L3.6mm_D1.6mm_P7.62mm_Horizontal -> Resistor_THT:R_Axial_DIN0204_L3.6mm_D1.6mm_P5.08mm_Horizontal
Changed lines of the file:
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@@
 			)
 		)
-		(property "Footprint" "Resistor_THT:R_Axial_DIN0204_L3.6mm_D1.6mm_P7.62mm_Horizontal"
+		(property "Footprint" "Resistor_THT:R_Axial_DIN0204_L3.6mm_D1.6mm_P5.08mm_Horizontal"
 			(at 144.78 102.362 90)
 			(effects
@@
 			)
 		)
-		(property "Footprint" "Resistor_THT:R_Axial_DIN0204_L3.6mm_D1.6mm_P7.62mm_Horizontal"
+		(property "Footprint" "Resistor_SMD:R_0805_2012Metric_Pad1.20x1.40mm_HandSolder"
 			(at 109.728 99.06 90)
 			(effects
@@
 			)
 		)
-		(property "Mouser part no." " 603-MFR-12FTF52-27K"
+		(property "Mouser part no." " 603-RE0805FRE0727KL"
 			(at 107.95 99.06 0)
 			(effects
