File: board/osborne-floppy-emulator.kicad_pcb (KiCad board)
At the start: 2 copper layers, 77.6 x 90.8 mm, 68 parts, among them J1 Connector Out, J2 USB_A, J3 SWD Connector, J4 Connector In, Q1 BC557, Q2 BC547, Q3 T2N7002BK, Q4 BC847C, Q5 BC847C, Q6 BC847C, Q7 BC847C, Q8 BC847C, Q9 BC847C, U1 W25Q16JVSSIM, U2 RP2040, U3 TL494

Commit message: add TPs for the extra pins to the board
Parts:
- added TP10: TestPoint, TestPoint:TestPoint_Pad_D1.0mm, B.Cu at (131.7, 78.8)
- added TP11: TestPoint, TestPoint:TestPoint_Pad_D1.0mm, B.Cu at (131.7, 76.7)
- added TP12: TestPoint, TestPoint:TestPoint_Pad_D1.0mm, F.Cu at (131.7, 76.8)
- added TP13: TestPoint, TestPoint:TestPoint_Pad_D1.0mm, F.Cu at (133.8, 76.8)
- added TP14: TestPoint, TestPoint:TestPoint_Pad_D1.0mm, B.Cu at (130.3, 74.8)
- added TP15: TestPoint, TestPoint:TestPoint_Pad_D1.0mm, B.Cu at (130.3, 72.7)
- added TP16: TestPoint, TestPoint:TestPoint_Pad_D1.0mm, B.Cu at (134.4, 71.5)
- added TP17: TestPoint, TestPoint:TestPoint_Pad_D1.0mm, B.Cu at (132.3, 71.5)
- added TP4: TestPoint, TestPoint:TestPoint_Pad_D1.0mm, F.Cu at (134.4, 69.8)
- added TP5: TestPoint, TestPoint:TestPoint_Pad_D1.0mm, F.Cu at (136.6, 69.8)
- added TP6: TestPoint, TestPoint:TestPoint_Pad_D1.0mm, F.Cu at (134.4, 72.3)
- added TP7: TestPoint, TestPoint:TestPoint_Pad_D1.0mm, F.Cu at (136.6, 72.3)
- added TP8: TestPoint, TestPoint:TestPoint_Pad_D1.0mm, B.Cu at (127.2, 78.8)
- added TP9: TestPoint, TestPoint:TestPoint_Pad_D1.0mm, B.Cu at (127.2, 76.7)
- moved C11 0.18 mm to (132.5, 74.7)
Routing:
- net Net-(U2-GPIO22): track 0.00 -> 9.58 mm, vias 0 -> 1
- net Net-(U2-GPIO23): track 0.00 -> 8.88 mm, vias 0 -> 1
- net Net-(U2-GPIO28_ADC2): track 0.00 -> 7.76 mm
- net Net-(U2-GPIO27_ADC1): track 0.00 -> 7.63 mm
- net Net-(U2-GPIO24): track 0.00 -> 6.01 mm, vias 0 -> 1
- net Net-(U2-GPIO29_ADC3): track 0.00 -> 5.42 mm
- net Net-(U2-GPIO26_ADC0): track 0.00 -> 5.34 mm
- net Net-(U2-GPIO21): track 0.00 -> 5.13 mm
- net Net-(U2-GPIO25): track 0.00 -> 4.48 mm, vias 0 -> 1
- net Net-(U2-GPIO18): track 0.00 -> 3.95 mm, vias 0 -> 1
- net Net-(U2-GPIO16): track 0.00 -> 3.85 mm, vias 0 -> 1
- net Net-(U2-GPIO20): track 0.00 -> 3.22 mm
- net GND: track 31.3 -> 28.1 mm
- net Net-(U2-GPIO19): track 0.00 -> 2.86 mm, vias 0 -> 1
- net Net-(U2-GPIO17): track 0.00 -> 2.66 mm, vias 0 -> 1

Commit message: connect power
Parts:
- Cout2, L2, R1: moved to F.Cu
- moved Cout2 6.31 mm to (145.3, 73.4)
- moved J2 6.01 mm to (129.6, 52.3)
- moved R1 5.90 mm to (112.0, 104.0), turned to 0 degrees
- moved L2 4.80 mm to (148.3, 73.2), turned to 90 degrees
- moved C10 0.25 mm to (119.8, 74.5), turned to 15 degrees
Routing:
- net +5V: track 5.51 -> 133.0 mm, vias 0 -> 7
- net +3V3: track 30.9 -> 137.3 mm, vias 0 -> 8
- net +12V: track 26.6 -> 128.8 mm, vias 1 -> 5
- net /Connector/-0V: track 22.3 -> 106.2 mm, vias 0 -> 11
- net GND: track 28.1 -> 50.0 mm, vias 7 -> 12
- net /Processor/Port D-: track 0.00 -> 4.06 mm
- net /Processor/Port D+: track 0.00 -> 4.06 mm
- net Net-(Q8-B): track 0.00 -> 2.33 mm
- added copper zone on F.Cu, net +12V
- added copper zone on F.Cu, net +5V
- added copper zone on B.Cu, net /Connector/-0V
- added copper zone on B.Cu, net GND
Other:
- board size 77.6 x 90.8 mm -> 77.6 x 93.2 mm
