File: board/osborne-floppy-emulator.kicad_pcb (KiCad board)
At the start: 2 copper layers, 77.6 x 93.2 mm, 82 parts, among them J1 Connector Out, J2 USB_A, J3 SWD Connector, J4 Connector In, Q1 BC557, Q2 BC547, Q3 T2N7002BK, Q4 BC847C, Q5 BC847C, Q6 BC847C, Q7 BC847C, Q8 BC847C, Q9 BC847C, U1 W25Q16JVSSIM, U2 RP2040, U3 TL494

Commit message: fix board borders and modify ground plane
Other:
- board size 77.6 x 93.2 mm -> 61.6 x 54 mm
Changed lines of the file:
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@@
 	)
 	(gr_rect
-		(start 90.4 14.8)
-		(end 168 108)
+		(start 90.4 53)
+		(end 152 106.95)
 		(stroke
 			(width 0.05)
@@
 		(polygon
 			(pts
-				(xy 152.5 59.75) (xy 102.7 59.75) (xy 102.65 105.1) (xy 152.45 105.1)
+				(xy 152 53) (xy 102.7 53) (xy 102.65 106.95) (xy 152 106.95)
 			)
 		)
@@
 			(pts
 				(xy 96.6 60.3) (xy 96.6 73.75) (xy 92 73.75) (xy 92 83.4) (xy 96.6 83.4) (xy 96.6 86.5) (xy 92 86.5)
-				(xy 92 93.55) (xy 96.6 93.55) (xy 96.6 105.1) (xy 90.7 105.1) (xy 90.7 60.3)
+				(xy 92 93.55) (xy 96.6 93.55) (xy 96.6 105.1) (xy 90.9 105.05) (xy 90.9 60.3)
 			)
 		)

Commit message: move more of the +3V3 line to the front
Parts:
- moved R2 1.11 mm to (125.6, 92.1), turned to 15 degrees
- moved J3 0.10 mm to (124.6, 86.8)
Routing:
- net +3V3: track 137.3 -> 133.3 mm, vias 8 -> 9
- net Net-(Q2-B): track 29.7 -> 28.3 mm
- net Net-(Q1-B): track 8.17 -> 9.03 mm
- net +12V: track 128.8 -> 129.4 mm

Commit message: move silkscreen text
Other:
- board text added: "Osborne 1 FDD emulator v. 2 r. A"
- board text removed: "Osborne 1 FDD emulator v. 1 r. A"
Changed lines of the file:
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@@
 	)
 	(gr_text "JLCJLCJLCJLC"
-		(at 165.2 17.677806 90)
+		(at 101.65 55.6 0)
 		(layer "B.SilkS")
 		(effects
@@
 		)
 	)
-	(gr_text "Osborne 1\nFDD emulator\nv. 1 r. A"
-		(at 164.8 34 90)
+	(gr_text "Osborne 1\nFDD emulator\nv. 2 r. A"
+		(at 103.15 60.3 0)
 		(layer "F.SilkS")
 		(effects

Commit message: shrink board slightly
Parts:
- moved R11 0.25 mm to (131.7, 93.9)
Other:
- board size 61.6 x 54 mm -> 61.6 x 53.7 mm
Changed lines of the file:
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@@
 	(footprint "Resistor_THT:R_Axial_DIN0207_L6.3mm_D2.5mm_P10.16mm_Horizontal"
 		(layer "B.Cu")
-		(at 131.7 94.12 -90)
+		(at 131.7 93.87 -90)
 		(descr "Resistor, Axial_DIN0207 series, Axial, Horizontal, pin pitch=10.16mm, 0.25W = 1/4W, length*diameter=6.3*2.5mm^2, http://cdn-reichelt.de/documents/datenblatt/B400/1_4W%23YAG.pdf")
 		(tags "Resistor Axial_DIN0207 series Axial Horizontal pin pitch 10.16mm 0.25W = 1/4W length 6.3mm diameter 2.5mm")
@@
 	(gr_rect
 		(start 90.4 53)
-		(end 152 106.95)
+		(end 152 106.65)
 		(stroke
 			(width 0.05)
@@
 	)
 	(segment
-		(start 132.3125 99.2625)
-		(end 131.7 104.279999)
+		(start 126.175 98.225)
+		(end 125.4 98.275)
 		(width 0.4)
 		(layer "F.Cu")
@@
 	)
 	(segment
-		(start 126.175 98.225)
-		(end 125.4 98.275)
+		(start 127.5 98.3)
+		(end 132.3125 99.2625)
 		(width 0.4)
 		(layer "F.Cu")
@@
 	)
 	(segment
-		(start 127.5 98.3)
-		(end 132.3125 99.2625)
+		(start 132.3125 99.2625)
+		(end 131.7 104.03)
 		(width 0.4)
 		(layer "F.Cu")
@@
 	(segment
 		(start 132.3125 97.5375)
-		(end 131.7 94.12)
+		(end 131.7 93.87)
 		(width 0.4)
 		(layer "F.Cu")
@@
 	)
 	(segment
-		(start 91.4 103.75)
-		(end 91.4 93.9)
-		(width 1)
-		(layer "F.Cu")
-		(net 11)
-	)
-	(segment
-		(start 148.2 101.55)
-		(end 143.45 104.75)
+		(start 91.75 104.85)
+		(end 91.4 103.75)
 		(width 1)
 		(layer "F.Cu")
@@
 	)
 	(segment
-		(start 143.2 83)
-		(end 145.700001 83)
+		(start 91.4 103.75)
+		(end 91.4 93.9)
 		(width 1)
 		(layer "F.Cu")
@@
 	)
 	(segment
-		(start 151 88.5)
-		(end 151 96.7)
+		(start 143.2 83)
+		(end 145.700001 83)
 		(width 1)
 		(layer "F.Cu")
@@
 	)
 	(segment
-		(start 146.099999 88.5)
-		(end 147.8 88.5)
+		(start 151 96.7)
+		(end 148.2 101.55)
 		(width 1)
 		(layer "F.Cu")
@@
 	)
 	(segment
-		(start 91.75 104.85)
-		(end 91.4 103.75)
+		(start 148.2 101.55)
+		(end 143.45 104.75)
 		(width 1)
 		(layer "F.Cu")
@@
 	)
 	(segment
-		(start 135 105.95)
-		(end 105.4 105.8)
+		(start 146.099999 88.5)
+		(end 147.8 88.5)
 		(width 1)
 		(layer "F.Cu")
@@
 	)
 	(segment
-		(start 105.4 105.8)
-		(end 93 105.65)
+		(start 142.5 82.6)
+		(end 143.2 83)
 		(width 1)
 		(layer "F.Cu")
@@
 	)
 	(segment
-		(start 151 96.7)
-		(end 148.2 101.55)
+		(start 139.8 62.85)
+		(end 140.75 63.15)
 		(width 1)
 		(layer "F.Cu")
@@
 	)
 	(segment
-		(start 143.45 104.75)
-		(end 135 105.95)
+		(start 137.15 63.25)
+		(end 135.6 63.026923)
 		(width 1)
 		(layer "F.Cu")
@@
 	)
 	(segment
-		(start 142.5 82.6)
-		(end 143.2 83)
+		(start 141.9 64.9)
+		(end 142 70.35)
 		(width 1)
 		(layer "F.Cu")
@@
 	)
 	(segment
-		(start 93 105.65)
-		(end 91.75 104.85)
+		(start 141.5 64.1)
+		(end 141.9 64.9)
 		(width 1)
 		(layer "F.Cu")
@@
 	)
 	(segment
-		(start 139.8 62.85)
-		(end 140.75 63.15)
+		(start 93 105.65)
+		(end 91.75 104.85)
 		(width 1)
 		(layer "F.Cu")
@@
 	)
 	(segment
-		(start 137.15 63.25)
-		(end 135.6 63.026923)
+		(start 135 105.65)
+		(end 93 105.65)
 		(width 1)
 		(layer "F.Cu")
@@
 	)
 	(segment
-		(start 141.9 64.9)
-		(end 142 70.35)
+		(start 143.45 104.75)
+		(end 135 105.65)
 		(width 1)
 		(layer "F.Cu")
@@
 	)
 	(segment
-		(start 141.5 64.1)
-		(end 141.9 64.9)
+		(start 135.6 63.026923)
+		(end 134.25 61.9)
 		(width 1)
 		(layer "F.Cu")
@@
 	)
 	(segment
-		(start 135.6 63.026923)
-		(end 134.25 61.9)
+		(start 151 88.5)
+		(end 151 96.7)
 		(width 1)
 		(layer "F.Cu")
@@
 	)
 	(segment
-		(start 125.05 90.9)
-		(end 126.6 90.95)
-		(width 0.4)
-		(layer "F.Cu")
-		(net 50)
-	)
-	(segment
-		(start 126.6 90.95)
-		(end 127.65 91.3)
+		(start 121.3 95.6)
+		(end 121.8 95.4)
 		(width 0.4)
 		(layer "F.Cu")
@@
 	)
 	(segment
-		(start 136.2 95.1)
-		(end 141.499556 95.405)
+		(start 130.8 92)
+		(end 132.5 92.7)
 		(width 0.4)
 		(layer "F.Cu")
@@
 	)
 	(segment
-		(start 127.65 91.3)
-		(end 130.8 92)
+		(start 125.05 90.9)
+		(end 126.6 90.95)
 		(width 0.4)
 		(layer "F.Cu")
@@
 	)
 	(segment
-		(start 124.1 91.3)
-		(end 125.05 90.9)
+		(start 132.5 92.7)
+		(end 133.8 93.9)
 		(width 0.4)
 		(layer "F.Cu")
@@
 	)
 	(segment
-		(start 120.45 95.625)
-		(end 121.3 95.6)
+		(start 127.65 91.3)
+		(end 130.8 92)
 		(width 0.4)
 		(layer "F.Cu")
@@
 	)
 	(segment
-		(start 121.8 95.4)
-		(end 122.4 94)
+		(start 120.45 95.625)
+		(end 121.3 95.6)
 		(width 0.4)
 		(layer "F.Cu")
@@
 	)
 	(segment
-		(start 132.4 92.9)
-		(end 133.8 94.1)
+		(start 123.1 92.4)
+		(end 124.1 91.3)
 		(width 0.4)
 		(layer "F.Cu")
@@
 	)
 	(segment
-		(start 122.4 94)
-		(end 123.1 92.4)
+		(start 126.6 90.95)
+		(end 127.65 91.3)
 		(width 0.4)
 		(layer "F.Cu")
@@
 	)
 	(segment
-		(start 133.8 94.1)
-		(end 136.2 95.1)
+		(start 136.2 95.1)
+		(end 141.499556 95.405)
 		(width 0.4)
 		(layer "F.Cu")
@@
 	)
 	(segment
-		(start 121.3 95.6)
-		(end 121.8 95.4)
+		(start 121.8 95.4)
+		(end 122.4 94)
 		(width 0.4)
 		(layer "F.Cu")
@@
 	)
 	(segment
-		(start 130.8 92)
-		(end 132.4 92.9)
+		(start 122.4 94)
+		(end 123.1 92.4)
 		(width 0.4)
 		(layer "F.Cu")
@@
 	)
 	(segment
-		(start 123.1 92.4)
-		(end 124.1 91.3)
+		(start 133.8 93.9)
+		(end 136.2 95.1)
 		(width 0.4)
 		(layer "F.Cu")
@@
 	)
 	(segment
-		(start 136.4 91.4)
-		(end 136.2 90.7)
+		(start 124.1 91.3)
+		(end 125.05 90.9)
+		(width 0.4)
+		(layer "F.Cu")
+		(net 50)
+	)
+	(segment
+		(start 132.980178 90.1639)
+		(end 133.4 92.1)
 		(width 0.6)
 		(layer "F.Cu")
@@
 	)
 	(segment
-		(start 133.3 92.2)
-		(end 134.3 93.1)
+		(start 136 93.1)
+		(end 136.5 92.3)
 		(width 0.6)
 		(layer "F.Cu")
@@
 	)
 	(segment
-		(start 134.3 93.1)
-		(end 135.3 93.4)
+		(start 133.4 92.1)
+		(end 134.25 92.9)
 		(width 0.6)
 		(layer "F.Cu")
@@
 	)
 	(segment
-		(start 136.2 90.7)
-		(end 136.373273 89.4713)
+		(start 136.4 91.4)
+		(end 136.2 90.7)
 		(width 0.6)
 		(layer "F.Cu")
@@
 	)
 	(segment
-		(start 132.980178 90.1639)
-		(end 133.3 92.2)
+		(start 134.25 92.9)
+		(end 135.3 93.4)
 		(width 0.6)
 		(layer "F.Cu")
@@
 	)
 	(segment
-		(start 136 93.1)
-		(end 136.5 92.3)
+		(start 136.2 90.7)
+		(end 136.373273 89.4713)
 		(width 0.6)
 		(layer "F.Cu")
@@
 		(polygon
 			(pts
-				(xy 152 53) (xy 102.7 53) (xy 102.65 106.95) (xy 152 106.95)
+				(xy 152 53) (xy 102.7 53) (xy 102.65 106.65) (xy 152 106.65)
 			)
 		)

Commit message: add power pin to debug connector
Parts:
- J3: footprint Connector_PinSocket_2.54mm:PinSocket_1x03_P2.54mm_Vertical -> Connector_PinSocket_2.54mm:PinSocket_1x04_P2.54mm_Vertical
- moved J3 2.55 mm to (122.0, 86.8)
Connections:
- J3 pad 1: GND -> +3V3
- J3 pad 2: /Processor/Debug clock -> GND
- J3 pad 3: /Processor/Debug data -> /Processor/Debug clock
Routing:
- net +3V3: track 133.3 -> 132.7 mm
Changed lines of the file:
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@@
 		)
 	)
-	(footprint "Connector_PinSocket_2.54mm:PinSocket_1x03_P2.54mm_Vertical"
+	(footprint "Connector_PinSocket_2.54mm:PinSocket_1x04_P2.54mm_Vertical"
 		(layer "F.Cu")
-		(at 124.6 86.8 90)
-		(descr "Through hole straight socket strip, 1x03, 2.54mm pitch, single row (from Kicad 4.0.7), script generated")
-		(tags "Through hole socket strip THT 1x03 2.54mm single row")
+		(at 122.05 86.8 90)
+		(descr "Through hole straight socket strip, 1x04, 2.54mm pitch, single row (from Kicad 4.0.7), script generated")
+		(tags "Through hole socket strip THT 1x04 2.54mm single row")
 		(property "Reference" "J3"
 			(at 0 -2.77 90)
@@
 		)
 		(property "Value" "SWD Connector"
-			(at 0 7.85 90)
+			(at 0 10.39 90)
 			(layer "F.Fab")
 			(effects
@@
 			)
 		)
-		(property "Footprint" "Connector_PinSocket_2.54mm:PinSocket_1x03_P2.54mm_Vertical"
+		(property "Footprint" "Connector_PinSocket_2.54mm:PinSocket_1x04_P2.54mm_Vertical"
 			(at 0 0 90)
 			(unlocked yes)
@@
 			)
 		)
-		(property "Description" "Generic connector, single row, 01x03, script generated"
+		(property "Description" "Generic connector, single row, 01x04, script generated"
 			(at 0 0 90)
 			(unlocked yes)
@@
 		(fp_line
 			(start 1.33 1.27)
-			(end 1.33 6.41)
+			(end 1.33 8.95)
 			(stroke
 				(width 0.12)
@@
 		(fp_line
 			(start -1.33 1.27)
-			(end -1.33 6.41)
+			(end -1.33 8.95)
 			(stroke
 				(width 0.12)
@@
 		)
 		(fp_line
-			(start -1.33 6.41)
-			(end 1.33 6.41)
+			(start -1.33 8.95)
+			(end 1.33 8.95)
 			(stroke
 				(width 0.12)
@@
 		(fp_line
 			(start 1.75 -1.8)
-			(end 1.75 6.85)
+			(end 1.75 9.4)
 			(stroke
 				(width 0.05)
@@
 		)
 		(fp_line
-			(start 1.75 6.85)
-			(end -1.8 6.85)
+			(start 1.75 9.4)
+			(end -1.8 9.4)
 			(stroke
 				(width 0.05)
@@
 		)
 		(fp_line
-			(start -1.8 6.85)
+			(start -1.8 9.4)
 			(end -1.8 -1.8)
 			(stroke
@@
 		(fp_line
 			(start 1.27 -0.635)
-			(end 1.27 6.35)
+			(end 1.27 8.89)
 			(stroke
 				(width 0.1)
@@
 		)
 		(fp_line
-			(start 1.27 6.35)
-			(end -1.27 6.35)
+			(start 1.27 8.89)
+			(end -1.27 8.89)
 			(stroke
 				(width 0.1)
@@
 		)
 		(fp_line
-			(start -1.27 6.35)
+			(start -1.27 8.89)
 			(end -1.27 -1.27)
 			(stroke
@@
 		)
 		(fp_text user "${REFERENCE}"
-			(at 0 2.54 180)
+			(at 0 3.81 180)
 			(layer "F.Fab")
 			(effects
@@
 			(layers "*.Cu" "*.Mask")
 			(remove_unused_layers no)
-			(net 5 "GND")
+			(net 9 "+3V3")
 			(pinfunction "Pin_1")
 			(pintype "passive")
@@
 			(layers "*.Cu" "*.Mask")
 			(remove_unused_layers no)
-			(net 44 "/Processor/Debug clock")
+			(net 5 "GND")
 			(pinfunction "Pin_2")
 			(pintype "passive")
@@
 			(layers "*.Cu" "*.Mask")
 			(remove_unused_layers no)
-			(net 43 "/Processor/Debug data")
+			(net 44 "/Processor/Debug clock")
 			(pinfunction "Pin_3")
 			(pintype "passive")
 		)
-		(model "${KICAD8_3DMODEL_DIR}/Connector_PinSocket_2.54mm.3dshapes/PinSocket_1x03_P2.54mm_Vertical.wrl"
+		(pad "4" thru_hole oval
+			(at 0 7.62 90)
+			(size 1.7 1.7)
+			(drill 1)
+			(layers "*.Cu" "*.Mask")
+			(remove_unused_layers no)
+			(net 43 "/Processor/Debug data")
+			(pinfunction "Pin_4")
+			(pintype "passive")
+		)
+		(model "${KICAD8_3DMODEL_DIR}/Connector_PinSocket_2.54mm.3dshapes/PinSocket_1x04_P2.54mm_Vertical.wrl"
 			(offset
 				(xyz 0 0 0)
@@
 		(fp_arc
 			(start 1.27 2.6)
-			(mid -1.132087 0.994977)
+			(mid -1.132087 0.994976)
 			(end -0.568477 -1.838478)
 			(stroke
@@
 		(fp_arc
 			(start 1.27 2.6)
-			(mid -1.132087 0.994977)
+			(mid -1.132087 0.994976)
 			(end -0.568477 -1.838478)
 			(stroke
@@
 	)
 	(segment
+		(start 124.59 86.8)
+		(end 124.6 83.9)
+		(width 0.4)
+		(layer "F.Cu")
+		(net 5)
+	)
+	(segment
 		(start 124.9 75.6)
 		(end 125.9 73.2)
@@
 	)
 	(segment
-		(start 124.6 86.8)
-		(end 124.6 83.9)
-		(width 0.4)
-		(layer "F.Cu")
-		(net 5)
-	)
-	(segment
-		(start 124.6 83.9)
-		(end 125.5 80.8625)
-		(width 0.4)
-		(layer "F.Cu")
-		(net 5)
-	)
-	(segment
 		(start 116.334808 65.558646)
 		(end 117.530358 64.954881)
@@
 	)
 	(segment
+		(start 124.6 83.9)
+		(end 125.5 80.8625)
+		(width 0.4)
+		(layer "F.Cu")
+		(net 5)
+	)
+	(segment
 		(start 124.65 96.55)
 		(end 125.05 96.9)
@@
 	)
 	(segment
-		(start 134.85 77.35)
-		(end 136 74)
-		(width 0.6)
-		(layer "F.Cu")
-		(net 9)
-	)
-	(segment
-		(start 131.65 87.6)
-		(end 132.2 85.95)
+		(start 132.75 80.15)
+		(end 133.55 78.7)
 		(width 0.6)
 		(layer "F.Cu")
@@
 	)
 	(segment
-		(start 133.55 78.7)
-		(end 134.15 78.1)
+		(start 131.65 87.6)
+		(end 132.2 85.95)
 		(width 0.6)
 		(layer "F.Cu")
@@
 	)
 	(segment
-		(start 121.2 82.8)
-		(end 121.2 87.25)
+		(start 132.65 82.35)
+		(end 132.75 80.15)
 		(width 0.6)
 		(layer "F.Cu")
@@
 	)
 	(segment
+		(start 121.2 82.8)
+		(end 122.05 86.8)
+		(width 0.6)
+		(layer "F.Cu")
+		(net 9)
+	)
+	(segment
 		(start 126.3 69.7625)
 		(end 126.3 68.6)
@@
 	)
 	(segment
-		(start 132.65 82.35)
-		(end 132.75 80.15)
-		(width 0.6)
-		(layer "F.Cu")
-		(net 9)
-	)
-	(segment
-		(start 127.3 88.45)
-		(end 130.45 88.2)
+		(start 134.85 77.35)
+		(end 136 74)
 		(width 0.6)
 		(layer "F.Cu")
@@
 	)
 	(segment
-		(start 132.2 85.95)
-		(end 132.65 82.35)
+		(start 122.05 86.8)
+		(end 122.5 88.2)
 		(width 0.6)
 		(layer "F.Cu")
@@
 	)
 	(segment
+		(start 123.55 88.65)
+		(end 127.3 88.45)
+		(width 0.6)
+		(layer "F.Cu")
+		(net 9)
+	)
+	(segment
 		(start 137.45 73.15)
 		(end 138.35 71.65)
@@
 	)
 	(segment
-		(start 132.75 80.15)
-		(end 133.55 78.7)
+		(start 133.55 78.7)
+		(end 134.15 78.1)
 		(width 0.6)
 		(layer "F.Cu")
@@
 	)
 	(segment
-		(start 134.15 78.1)
-		(end 134.85 77.35)
-		(width 0.6)
-		(layer "F.Cu")
-		(net 9)
-	)
-	(segment
 		(start 123.5 71)
 		(end 123.1 70.6)
@@
 	)
 	(segment
-		(start 121.2 87.25)
-		(end 121.95 88.25)
-		(width 0.6)
-		(layer "F.Cu")
-		(net 9)
-	)
-	(segment
 		(start 126.1 76.6375)
 		(end 126.1 78.4)
@@
 	)
 	(segment
-		(start 130.45 88.2)
-		(end 131.65 87.6)
-		(width 0.6)
+		(start 126.3 69.7625)
+		(end 126.5 69.7625)
+		(width 0.2)
 		(layer "F.Cu")
 		(net 9)
 	)
 	(segment
-		(start 126.3 69.7625)
-		(end 126.5 69.7625)
-		(width 0.2)
+		(start 127.3 88.45)
+		(end 130.45 88.2)
+		(width 0.6)
 		(layer "F.Cu")
 		(net 9)
@@
 	)
 	(segment
-		(start 123.4 88.55)
-		(end 127.3 88.45)
-		(width 0.6)
-		(layer "F.Cu")
-		(net 9)
-	)
-	(segment
 		(start 128.5 69.7625)
 		(end 128.5 70.25)
@@
 	)
 	(segment
+		(start 132.2 85.95)
+		(end 132.65 82.35)
+		(width 0.6)
+		(layer "F.Cu")
+		(net 9)
+	)
+	(segment
 		(start 136.6 73.7)
 		(end 137.45 73.15)
@@
 	)
 	(segment
+		(start 122.5 88.2)
+		(end 123.55 88.65)
+		(width 0.6)
+		(layer "F.Cu")
+		(net 9)
+	)
+	(segment
 		(start 126.1 78.4)
 		(end 125.5 79.1375)
@@
 	)
 	(segment
+		(start 130.45 88.2)
+		(end 131.65 87.6)
+		(width 0.6)
+		(layer "F.Cu")
+		(net 9)
+	)
+	(segment
 		(start 120.95 66.3)
 		(end 119.55 59.3)
@@
 	)
 	(segment
-		(start 121.95 88.25)
-		(end 123.4 88.55)
+		(start 134.15 78.1)
+		(end 134.85 77.35)
 		(width 0.6)
 		(layer "F.Cu")
@@
 	(segment
 		(start 130.3 83.5)
-		(end 129.68 86.8)
+		(end 129.67 86.8)
 		(width 0.2)
 		(layer "F.Cu")
@@
 	)
 	(segment
+		(start 127.2 83.5)
+		(end 127.13 86.8)
+		(width 0.2)
+		(layer "F.Cu")
+		(net 44)
+	)
+	(segment
 		(start 127.2 78.1)
 		(end 127.8 78.5)
@@
 		(width 0.2)
 		(layer "F.Cu")
-		(net 44)
-	)
-	(segment
-		(start 127.2 83.5)
-		(end 127.14 86.8)
-		(width 0.2)
-		(layer "F.Cu")

Commit message: make pads on rp2040 footprint extra long
Parts:
- U2: footprint Package_DFN_QFN:QFN-56-1EP_7x7mm_P0.4mm_EP3.2x3.2mm -> custom-footprints:QFN-56_EP_7x7_Pitch0.4mm_Extralong
- moved C10 0.74 mm to (119.2, 74.9), turned to 30 degrees
- moved C9 0.43 mm to (132.1, 69.5)
- moved C13 0.42 mm to (126.8, 80.3)
- moved C8 0.38 mm to (119.7, 69.8)
- moved C7 0.30 mm to (131.5, 67.7)
- moved C6 0.28 mm to (131.5, 65.7)
- moved TP4 0.28 mm to (134.7, 69.8)
- moved TP5 0.27 mm to (136.8, 69.8)
- moved C12 0.21 mm to (125.3, 80.0)
- moved TP1 0.18 mm to (130.4, 79.2)
- moved C11 0.15 mm to (132.7, 74.7)
Routing:
- net +3V3: track 132.7 -> 133.9 mm
- net GND: track 49.9 -> 48.8 mm
- net Net-(U2-VREG_VOUT): track 18.5 -> 19.4 mm
