File: board/connector.kicad_sch (KiCad schematic)
At the start: 4 parts, among them J1 Connector Out, J4 Connector In, Q5 BC847C, Q6 BC847C

Commit message: fix connector in part number (so expensive ):
Parts:
- J4: Mouser part no. 710-61304021821 -> 855-M20-7872042
Changed lines of the file:
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@@
 			)
 		)
-		(property "Mouser part no." " 710-61304021821"
+		(property "Mouser part no." "855-M20-7872042"
 			(at 156.21 82.55 0)
 			(effects

Commit message: fix BOM, add column for mfr. part number
Parts:
- J1: Mouser part no. 855-M20-7812045 -> 855-M20-7812045; Part no. (none) -> M20-7812045
- J4: Part no. (none) -> M20-7872042
- Q5, Q6: Mouser part no. 771-BC847C-T/R -> 771-BC847C-T/R; Part no. (none) -> BC847C-T/R
Changed lines of the file:
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@@
+			)
+		)
+		(property "Part no." "M20-7872042"
+			(at 156.21 82.55 0)
+			(effects
+				(font
+					(size 1.27 1.27)
+				)
+				(hide yes)
 			)
 		)
@@
 			)
 		)
-		(property "Mouser part no." " 771-BC847C-T/R"
+		(property "Mouser part no." "771-BC847C-T/R"
+			(at 186.69 121.92 0)
+			(effects
+				(font
+					(size 1.27 1.27)
+				)
+				(hide yes)
+			)
+		)
+		(property "Part no." "BC847C-T/R"
 			(at 186.69 121.92 0)
 			(effects
@@
 			)
 		)
-		(property "Mouser part no." " 855-M20-7812045"
+		(property "Mouser part no." "855-M20-7812045"
+			(at 156.21 134.62 0)
+			(effects
+				(font
+					(size 1.27 1.27)
+				)
+				(hide yes)
+			)
+		)
+		(property "Part no." "M20-7812045"
 			(at 156.21 134.62 0)
 			(effects
@@
 			)
 		)
-		(property "Mouser part no." " 771-BC847C-T/R"
+		(property "Mouser part no." "771-BC847C-T/R"
 			(at 205.74 124.46 0)
 			(effects
+				(font
+					(size 1.27 1.27)
+				)
+				(hide yes)
+			)
+		)
+		(property "Part no." "BC847C-T/R"
+			(at 205.74 124.46 0)
+			(effects

Commit message: change 2x17 connector part numbers to ones available at LCSC
Parts:
- J1: Part no. M20-7812045 -> PZ254-2-17-S
- J4: Part no. M20-7872042 -> FH-00357
Changed lines of the file:
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@@
 			)
 		)
-		(property "Part no." "M20-7872042"
+		(property "Part no." "FH-00357"
 			(at 156.21 82.55 0)
 			(effects
@@
 			)
 		)
-		(property "Part no." "M20-7812045"
-			(at 156.21 134.62 0)
-			(effects
+		(property "Part no." "PZ254-2-17-S"
+			(at 156.21 134.62 0)
+			(effects

Commit message: fix BOM, add more LCSC part numbers
Parts:
- J1: LCSC part no. (none) -> C3294475
- J4: LCSC part no. (none) -> C2685114
- Q5, Q6: LCSC part no. (none) -> C181141
Changed lines of the file:
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@@
+			)
+		)
+		(property "LCSC part no." "C2685114"
+			(at 156.21 82.55 0)
+			(effects
+				(font
+					(size 1.27 1.27)
+				)
+				(hide yes)
 			)
 		)
@@
 			)
 		)
+		(property "LCSC part no." "C181141"
+			(at 186.69 121.92 0)
+			(effects
+				(font
+					(size 1.27 1.27)
+				)
+				(hide yes)
+			)
+		)
 		(pin "3"
 		)
@@
 			)
 		)
+		(property "LCSC part no." "C3294475"
+			(at 156.21 134.62 0)
+			(effects
+				(font
+					(size 1.27 1.27)
+				)
+				(hide yes)
+			)
+		)
 		(pin "2"
 		)
@@
 			(at 205.74 124.46 0)
 			(effects
+				(font
+					(size 1.27 1.27)
+				)
+				(hide yes)
+			)
+		)
+		(property "LCSC part no." "C181141"
+			(at 205.74 124.46 0)
+			(effects
