File: board/osborne-floppy-emulator.kicad_sch (KiCad schematic)
At the start: 2 parts, among them J2 USB_A, J3 SWD Connector

Commit message: add power pin to debug connector
Parts:
- J3: footprint Connector_PinSocket_2.54mm:PinSocket_1x03_P2.54mm_Vertical -> Connector_PinSocket_2.54mm:PinSocket_1x04_P2.54mm_Vertical; symbol Connector:Conn_01x03_Socket -> Connector:Conn_01x04_Socket
Connections:
- net GND: now also J3.2 (Pin_2); no longer J3.1 (Pin_1)
- net Processor/Debug clock: now also J3.3 (Pin_3); no longer J3.2 (Pin_2)
- net Processor/Debug data: now also J3.4 (Pin_4); no longer J3.3 (Pin_3)
- new net +3V3: J3.1 (Pin_1)
Changed lines of the file:
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@@
 	(wire
 		(pts
-			(xy 73.66 137.16) (xy 72.39 137.16)
+			(xy 74.93 137.16) (xy 72.39 137.16)
 		)
 		(stroke
@@
 	(wire
 		(pts
+			(xy 73.66 139.7) (xy 73.66 130.81)
+		)
+		(stroke
+			(width 0)
+			(type default)
+		)
+	)
+	(wire
+		(pts
 			(xy 175.26 104.14) (xy 175.26 95.25)
 		)
@@
 	(wire
 		(pts
+			(xy 72.39 139.7) (xy 73.66 139.7)
+		)
+		(stroke
+			(width 0)
+			(type default)
+		)
+	)
+	(wire
+		(pts
 			(xy 59.69 104.14) (xy 59.69 105.41)
 		)
@@
 	(wire
 		(pts
-			(xy 73.66 138.43) (xy 73.66 137.16)
+			(xy 74.93 140.97) (xy 74.93 137.16)
 		)
 		(stroke
@@
 	(symbol
 		(lib_id "power:GND")
-		(at 73.66 138.43 0)
+		(at 74.93 140.97 0)
 		(unit 1)
 		(exclude_from_sim no)
@@
 		(fields_autoplaced yes)
 		(property "Reference" "#PWR030"
-			(at 73.66 144.78 0)
+			(at 74.93 147.32 0)
 			(effects
 				(font
@@
 		)
 		(property "Value" "GND"
-			(at 73.66 143.51 0)
+			(at 74.93 146.05 0)
 			(effects
 				(font
@@
 		)
 		(property "Footprint" ""
-			(at 73.66 138.43 0)
+			(at 74.93 140.97 0)
 			(effects
 				(font
@@
 		)
 		(property "Datasheet" ""
-			(at 73.66 138.43 0)
+			(at 74.93 140.97 0)
 			(effects
 				(font
@@
 		)
 		(property "Description" "Power symbol creates a global label with name \"GND\" , ground"
-			(at 73.66 138.43 0)
+			(at 74.93 140.97 0)
 			(effects
 				(font
@@
 				(path "/a407fcbc-6d86-4aa2-968f-b2fcdecb9640"
 					(reference "#PWR030")
+					(unit 1)
+				)
+			)
+		)
+	)
+	(symbol
+		(lib_id "power:+3V3")
+		(at 73.66 130.81 0)
+		(unit 1)
+		(exclude_from_sim no)
+		(in_bom yes)
+		(on_board yes)
+		(dnp no)
+		(fields_autoplaced yes)
+		(property "Reference" "#PWR032"
+			(at 73.66 134.62 0)
+			(effects
+				(font
+					(size 1.27 1.27)
+				)
+				(hide yes)
+			)
+		)
+		(property "Value" "+3V3"
+			(at 73.66 125.73 0)
+			(effects
+				(font
+					(size 1.27 1.27)
+				)
+			)
+		)
+		(property "Footprint" ""
+			(at 73.66 130.81 0)
+			(effects
+				(font
+					(size 1.27 1.27)
+				)
+				(hide yes)
+			)
+		)
+		(property "Datasheet" ""
+			(at 73.66 130.81 0)
+			(effects
+				(font
+					(size 1.27 1.27)
+				)
+				(hide yes)
+			)
+		)
+		(property "Description" "Power symbol creates a global label with name \"+3V3\""
+			(at 73.66 130.81 0)
+			(effects
+				(font
+					(size 1.27 1.27)
+				)
+				(hide yes)
+			)
+		)
+		(pin "1"
+		)
+		(instances
+			(project "osborne-floppy-emulator"
+				(path "/a407fcbc-6d86-4aa2-968f-b2fcdecb9640"
+					(reference "#PWR032")
 					(unit 1)
 				)
@@
 	)
 	(symbol
-		(lib_id "Connector:Conn_01x03_Socket")
-		(at 67.31 134.62 180)
+		(lib_id "Connector:Conn_01x04_Socket")
+		(at 67.31 137.16 180)
 		(unit 1)
 		(exclude_from_sim no)
@@
 		(dnp no)
 		(property "Reference" "J3"
-			(at 67.945 127 0)
+			(at 67.945 129.54 0)
 			(effects
 				(font
@@
 		)
 		(property "Value" "SWD Connector"
-			(at 67.945 129.54 0)
-			(effects
-				(font
-					(size 1.27 1.27)
-				)
-			)
-		)
-		(property "Footprint" "Connector_PinSocket_2.54mm:PinSocket_1x03_P2.54mm_Vertical"
-			(at 67.31 134.62 0)
+			(at 67.945 132.08 0)
+			(effects
+				(font
+					(size 1.27 1.27)
+				)
+			)
+		)
+		(property "Footprint" "Connector_PinSocket_2.54mm:PinSocket_1x04_P2.54mm_Vertical"
+			(at 67.31 137.16 0)
 			(effects
 				(font
@@
 		)
 		(property "Datasheet" "~"
-			(at 67.31 134.62 0)
-			(effects
-				(font
-					(size 1.27 1.27)
-				)
-				(hide yes)
-			)
-		)
-		(property "Description" "Generic connector, single row, 01x03, script generated"
-			(at 67.31 134.62 0)
+			(at 67.31 137.16 0)
+			(effects
+				(font
+					(size 1.27 1.27)
+				)
+				(hide yes)
+			)
+		)
+		(property "Description" "Generic connector, single row, 01x04, script generated"
+			(at 67.31 137.16 0)
 			(effects
 				(font
@@
 		)
 		(property "Mouser part no." " 737-RS1-03-G"
-			(at 67.31 134.62 0)
+			(at 67.31 137.16 0)
 			(effects
 				(font
@@
 		(pin "1"
 		)
+		(pin "4"
+		)
 		(instances

Commit message: fix part number for debug jumper
Parts:
- J3: Mouser part no. 737-RS1-03-G -> 737-RS1-04-G
Changed lines of the file:
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@@
 			)
 		)
-		(property "Mouser part no." " 737-RS1-03-G"
+		(property "Mouser part no." " 737-RS1-04-G"
 			(at 67.31 137.16 0)
 			(effects

Commit message: fix BOM, add column for mfr. part number
Parts:
- J2: Mouser part no. 737-USB-A-S-RA-SMT -> 737-USB-A-S-RA-SMT; Part no. (none) -> USB-A-S-RA-SMT
- J3: Mouser part no. 737-RS1-04-G -> 737-RS1-04-G; Part no. (none) -> S1-04-G
Changed lines of the file:
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@@
 			)
 		)
-		(property "Mouser part no." " 737-USB-A-S-RA-SMT"
+		(property "Mouser part no." "737-USB-A-S-RA-SMT"
+			(at 50.8 110.49 0)
+			(effects
+				(font
+					(size 1.27 1.27)
+				)
+				(hide yes)
+			)
+		)
+		(property "Part no." "USB-A-S-RA-SMT"
 			(at 50.8 110.49 0)
 			(effects
@@
 			)
 		)
-		(property "Mouser part no." " 737-RS1-04-G"
+		(property "Mouser part no." "737-RS1-04-G"
 			(at 67.31 137.16 0)
 			(effects
+				(font
+					(size 1.27 1.27)
+				)
+				(hide yes)
+			)
+		)
+		(property "Part no." "S1-04-G"
+			(at 67.31 137.16 0)
+			(effects

Commit message: fix BOM, add more LCSC part numbers
Parts:
- J2: LCSC part no. (none) -> C42644
- J3: LCSC part no. (none) -> C5116530
Changed lines of the file:
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@@
 			)
 		)
-		(property "Datasheet" " ~"
+		(property "Datasheet" "~"
 			(at 54.61 111.76 0)
 			(effects
@@
 		)
 		(property "Part no." "USB-A-S-RA-SMT"
+			(at 50.8 110.49 0)
+			(effects
+				(font
+					(size 1.27 1.27)
+				)
+				(hide yes)
+			)
+		)
+		(property "LCSC part no." "C42644"
 			(at 50.8 110.49 0)
 			(effects
@@
 			(at 67.31 137.16 0)
 			(effects
+				(font
+					(size 1.27 1.27)
+				)
+				(hide yes)
+			)
+		)
+		(property "LCSC part no." "C5116530"
+			(at 67.31 137.16 0)
+			(effects
