File: board/shifter.kicad_sch (KiCad schematic)
At the start: 20 parts, among them Q4 BC847C, Q7 BC847C, Q8 BC847C, Q9 BC847C

Commit message: fix BOM, add column for mfr. part number
Parts:
- D10, D11, D12, D2, D3, D4, D5, D6, D7, D8, D9: Mouser part no. 512-FDLL4148 -> 512-FDLL4148; Part no. (none) -> FDLL4148
- Q4, Q7, Q8, Q9: Mouser part no. 771-BC847C-T/R -> 771-BC847C-T/R; Part no. (none) -> BC847C-T/R
- R14, R16, R17, R18, R19: Mouser part no. 603-RE0805FRE0727KL -> 603-RE0805FRE0727KL; Part no. (none) -> RE0805FRE0727KL
Changed lines of the file:
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@@
 			)
 		)
-		(property "Mouser part no." " 603-RE0805FRE0727KL"
+		(property "Mouser part no." "603-RE0805FRE0727KL"
+			(at 146.05 99.06 0)
+			(effects
+				(font
+					(size 1.27 1.27)
+				)
+				(hide yes)
+			)
+		)
+		(property "Part no." "RE0805FRE0727KL"
 			(at 146.05 99.06 0)
 			(effects
@@
 			)
 		)
-		(property "Mouser part no." " 512-FDLL4148"
+		(property "Mouser part no." "512-FDLL4148"
+			(at 158.75 177.8 0)
+			(effects
+				(font
+					(size 1.27 1.27)
+				)
+				(hide yes)
+			)
+		)
+		(property "Part no." "FDLL4148"
 			(at 158.75 177.8 0)
 			(effects
@@
 			)
 		)
-		(property "Mouser part no." " 512-FDLL4148"
+		(property "Mouser part no." "512-FDLL4148"
+			(at 158.75 127 0)
+			(effects
+				(font
+					(size 1.27 1.27)
+				)
+				(hide yes)
+			)
+		)
+		(property "Part no." "FDLL4148"
 			(at 158.75 127 0)
 			(effects
@@
 			)
 		)
-		(property "Mouser part no." " 512-FDLL4148"
+		(property "Mouser part no." "512-FDLL4148"
+			(at 158.75 63.5 0)
+			(effects
+				(font
+					(size 1.27 1.27)
+				)
+				(hide yes)
+			)
+		)
+		(property "Part no." "FDLL4148"
 			(at 158.75 63.5 0)
 			(effects
@@
 			)
 		)
-		(property "Mouser part no." " 512-FDLL4148"
+		(property "Mouser part no." "512-FDLL4148"
+			(at 158.75 76.2 0)
+			(effects
+				(font
+					(size 1.27 1.27)
+				)
+				(hide yes)
+			)
+		)
+		(property "Part no." "FDLL4148"
 			(at 158.75 76.2 0)
 			(effects
@@
 			)
 		)
-		(property "Mouser part no." " 512-FDLL4148"
+		(property "Mouser part no." "512-FDLL4148"
+			(at 158.75 165.1 0)
+			(effects
+				(font
+					(size 1.27 1.27)
+				)
+				(hide yes)
+			)
+		)
+		(property "Part no." "FDLL4148"
 			(at 158.75 165.1 0)
 			(effects
@@
 			)
 		)
-		(property "Mouser part no." " 603-RE0805FRE0727KL"
+		(property "Mouser part no." "603-RE0805FRE0727KL"
+			(at 92.71 121.92 0)
+			(effects
+				(font
+					(size 1.27 1.27)
+				)
+				(hide yes)
+			)
+		)
+		(property "Part no." "RE0805FRE0727KL"
 			(at 92.71 121.92 0)
 			(effects
@@
 			)
 		)
-		(property "Mouser part no." " 512-FDLL4148"
+		(property "Mouser part no." "512-FDLL4148"
+			(at 158.75 114.3 0)
+			(effects
+				(font
+					(size 1.27 1.27)
+				)
+				(hide yes)
+			)
+		)
+		(property "Part no." "FDLL4148"
 			(at 158.75 114.3 0)
 			(effects
@@
 			)
 		)
-		(property "Mouser part no." " 603-RE0805FRE0727KL"
+		(property "Mouser part no." "603-RE0805FRE0727KL"
+			(at 92.71 146.05 0)
+			(effects
+				(font
+					(size 1.27 1.27)
+				)
+				(hide yes)
+			)
+		)
+		(property "Part no." "RE0805FRE0727KL"
 			(at 92.71 146.05 0)
 			(effects
@@
 			)
 		)
-		(property "Mouser part no." " 771-BC847C-T/R"
+		(property "Mouser part no." "771-BC847C-T/R"
+			(at 104.14 146.05 0)
+			(effects
+				(font
+					(size 1.27 1.27)
+				)
+				(hide yes)
+			)
+		)
+		(property "Part no." "BC847C-T/R"
 			(at 104.14 146.05 0)
 			(effects
@@
 			)
 		)
-		(property "Mouser part no." " 512-FDLL4148"
+		(property "Mouser part no." "512-FDLL4148"
+			(at 158.75 88.9 0)
+			(effects
+				(font
+					(size 1.27 1.27)
+				)
+				(hide yes)
+			)
+		)
+		(property "Part no." "FDLL4148"
 			(at 158.75 88.9 0)
 			(effects
@@
 			)
 		)
-		(property "Mouser part no." " 512-FDLL4148"
+		(property "Mouser part no." "512-FDLL4148"
+			(at 158.75 152.4 0)
+			(effects
+				(font
+					(size 1.27 1.27)
+				)
+				(hide yes)
+			)
+		)
+		(property "Part no." "FDLL4148"
 			(at 158.75 152.4 0)
 			(effects
@@
 			)
 		)
-		(property "Mouser part no." " 603-RE0805FRE0727KL"
+		(property "Mouser part no." "603-RE0805FRE0727KL"
+			(at 92.71 97.79 0)
+			(effects
+				(font
+					(size 1.27 1.27)
+				)
+				(hide yes)
+			)
+		)
+		(property "Part no." "RE0805FRE0727KL"
 			(at 92.71 97.79 0)
 			(effects
@@
 			)
 		)
-		(property "Mouser part no." " 603-RE0805FRE0727KL"
+		(property "Mouser part no." "603-RE0805FRE0727KL"
+			(at 92.71 73.66 0)
+			(effects
+				(font
+					(size 1.27 1.27)
+				)
+				(hide yes)
+			)
+		)
+		(property "Part no." "RE0805FRE0727KL"
 			(at 92.71 73.66 0)
 			(effects
@@
 			)
 		)
-		(property "Mouser part no." " 771-BC847C-T/R"
+		(property "Mouser part no." "771-BC847C-T/R"
+			(at 104.14 73.66 0)
+			(effects
+				(font
+					(size 1.27 1.27)
+				)
+				(hide yes)
+			)
+		)
+		(property "Part no." "BC847C-T/R"
 			(at 104.14 73.66 0)
 			(effects
@@
 			)
 		)
-		(property "Mouser part no." " 512-FDLL4148"
+		(property "Mouser part no." "512-FDLL4148"
+			(at 158.75 50.8 0)
+			(effects
+				(font
+					(size 1.27 1.27)
+				)
+				(hide yes)
+			)
+		)
+		(property "Part no." "FDLL4148"
 			(at 158.75 50.8 0)
 			(effects
@@
 			)
 		)
-		(property "Mouser part no." " 771-BC847C-T/R"
+		(property "Mouser part no." "771-BC847C-T/R"
+			(at 104.14 121.92 0)
+			(effects
+				(font
+					(size 1.27 1.27)
+				)
+				(hide yes)
+			)
+		)
+		(property "Part no." "BC847C-T/R"
 			(at 104.14 121.92 0)
 			(effects
@@
 			)
 		)
-		(property "Mouser part no." " 771-BC847C-T/R"
+		(property "Mouser part no." "771-BC847C-T/R"
+			(at 104.14 97.79 0)
+			(effects
+				(font
+					(size 1.27 1.27)
+				)
+				(hide yes)
+			)
+		)
+		(property "Part no." "BC847C-T/R"
 			(at 104.14 97.79 0)
 			(effects
@@
 			)
 		)
-		(property "Mouser part no." " 512-FDLL4148"
+		(property "Mouser part no." "512-FDLL4148"
+			(at 158.75 101.6 0)
+			(effects
+				(font
+					(size 1.27 1.27)
+				)
+				(hide yes)
+			)
+		)
+		(property "Part no." "FDLL4148"
 			(at 158.75 101.6 0)
 			(effects
@@
 			)
 		)
-		(property "Mouser part no." " 512-FDLL4148"
+		(property "Mouser part no." "512-FDLL4148"
 			(at 158.75 139.7 0)
 			(effects
+				(font
+					(size 1.27 1.27)
+				)
+				(hide yes)
+			)
+		)
+		(property "Part no." "FDLL4148"
+			(at 158.75 139.7 0)
+			(effects

Commit message: fix BOM, add more LCSC part numbers
Parts:
- D10, D11, D12, D2, D3, D4, D5, D6, D7, D8, D9: LCSC part no. (none) -> C78608
- Q4, Q7, Q8, Q9: LCSC part no. (none) -> C181141
- R14, R16, R17, R18, R19: LCSC part no. (none) -> C375523
Changed lines of the file:
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@@
+			)
+		)
+		(property "LCSC part no." "C375523"
+			(at 146.05 99.06 0)
+			(effects
+				(font
+					(size 1.27 1.27)
+				)
+				(hide yes)
 			)
 		)
@@
 			)
 		)
+		(property "LCSC part no." "C78608"
+			(at 158.75 177.8 0)
+			(effects
+				(font
+					(size 1.27 1.27)
+				)
+				(hide yes)
+			)
+		)
 		(pin "2"
 		)
@@
 			)
 		)
+		(property "LCSC part no." "C78608"
+			(at 158.75 127 0)
+			(effects
+				(font
+					(size 1.27 1.27)
+				)
+				(hide yes)
+			)
+		)
 		(pin "2"
 		)
@@
 			)
 		)
+		(property "LCSC part no." "C78608"
+			(at 158.75 63.5 0)
+			(effects
+				(font
+					(size 1.27 1.27)
+				)
+				(hide yes)
+			)
+		)
 		(pin "2"
 		)
@@
 			)
 		)
+		(property "LCSC part no." "C78608"
+			(at 158.75 76.2 0)
+			(effects
+				(font
+					(size 1.27 1.27)
+				)
+				(hide yes)
+			)
+		)
 		(pin "2"
 		)
@@
 			)
 		)
+		(property "LCSC part no." "C78608"
+			(at 158.75 165.1 0)
+			(effects
+				(font
+					(size 1.27 1.27)
+				)
+				(hide yes)
+			)
+		)
 		(pin "2"
 		)
@@
 			)
 		)
+		(property "LCSC part no." "C375523"
+			(at 92.71 121.92 0)
+			(effects
+				(font
+					(size 1.27 1.27)
+				)
+				(hide yes)
+			)
+		)
 		(pin "2"
 		)
@@
 			)
 		)
+		(property "LCSC part no." "C78608"
+			(at 158.75 114.3 0)
+			(effects
+				(font
+					(size 1.27 1.27)
+				)
+				(hide yes)
+			)
+		)
 		(pin "2"
 		)
@@
 			)
 		)
+		(property "LCSC part no." "C375523"
+			(at 92.71 146.05 0)
+			(effects
+				(font
+					(size 1.27 1.27)
+				)
+				(hide yes)
+			)
+		)
 		(pin "2"
 		)
@@
 			)
 		)
+		(property "LCSC part no." "C181141"
+			(at 104.14 146.05 0)
+			(effects
+				(font
+					(size 1.27 1.27)
+				)
+				(hide yes)
+			)
+		)
 		(pin "3"
 		)
@@
 			)
 		)
+		(property "LCSC part no." "C78608"
+			(at 158.75 88.9 0)
+			(effects
+				(font
+					(size 1.27 1.27)
+				)
+				(hide yes)
+			)
+		)
 		(pin "2"
 		)
@@
 			)
 		)
+		(property "LCSC part no." "C78608"
+			(at 158.75 152.4 0)
+			(effects
+				(font
+					(size 1.27 1.27)
+				)
+				(hide yes)
+			)
+		)
 		(pin "2"
 		)
@@
 			)
 		)
+		(property "LCSC part no." "C375523"
+			(at 92.71 97.79 0)
+			(effects
+				(font
+					(size 1.27 1.27)
+				)
+				(hide yes)
+			)
+		)
 		(pin "2"
 		)
@@
 			)
 		)
+		(property "LCSC part no." "C375523"
+			(at 92.71 73.66 0)
+			(effects
+				(font
+					(size 1.27 1.27)
+				)
+				(hide yes)
+			)
+		)
 		(pin "2"
 		)
@@
 			)
 		)
+		(property "LCSC part no." "C181141"
+			(at 104.14 73.66 0)
+			(effects
+				(font
+					(size 1.27 1.27)
+				)
+				(hide yes)
+			)
+		)
 		(pin "3"
 		)
@@
 			)
 		)
+		(property "LCSC part no." "C78608"
+			(at 158.75 50.8 0)
+			(effects
+				(font
+					(size 1.27 1.27)
+				)
+				(hide yes)
+			)
+		)
 		(pin "2"
 		)
@@
 			)
 		)
+		(property "LCSC part no." "C181141"
+			(at 104.14 121.92 0)
+			(effects
+				(font
+					(size 1.27 1.27)
+				)
+				(hide yes)
+			)
+		)
 		(pin "3"
 		)
@@
 			)
 		)
+		(property "LCSC part no." "C181141"
+			(at 104.14 97.79 0)
+			(effects
+				(font
+					(size 1.27 1.27)
+				)
+				(hide yes)
+			)
+		)
 		(pin "3"
 		)
@@
 			)
 		)
+		(property "LCSC part no." "C78608"
+			(at 158.75 101.6 0)
+			(effects
+				(font
+					(size 1.27 1.27)
+				)
+				(hide yes)
+			)
+		)
 		(pin "2"
 		)
@@
 			(at 158.75 139.7 0)
 			(effects
+				(font
+					(size 1.27 1.27)
+				)
+				(hide yes)
+			)
+		)
+		(property "LCSC part no." "C78608"
+			(at 158.75 139.7 0)
+			(effects
