File: board/regulator.kicad_sch (KiCad schematic)
At the start: 17 parts, among them Q1 BC557, Q2 BC547, U3 TL494

Commit message: fix BOM, add column for mfr. part number
Parts:
- C1: Mouser part no. 187-CL21A106KOQNNNE -> 187-CL21A106KOQNNNE; Part no. (none) -> CL21A106KOQNNNE
- C3: Mouser part no. 80-C0805C102J5G -> 80-C0805C102J5G; Part no. (none) -> C0805C102J5G
- C4: Mouser part no. 710-885012206095 -> 710-885012206095; Part no. (none) -> 885012206095
- Q1: Mouser part no. 637-BC557CBK -> 637-BC557CBK; Part no. (none) -> BC557CBK
- Q2: Mouser part no. 637-BC547CBK -> 637-BC547CBK; Part no. (none) -> BC547CBK
- R1: Mouser part no. 603-MFR-12FTF52-0R1 -> 603-MFR-12FTF52-0R1; Part no. (none) -> MFR-12FTF52-0R1
- R10: Mouser part no. 603-MFR-12FTF52-12K -> 603-MFR-12FTF52-12K; Part no. (none) -> MFR-12FTF52-12K
- R11: Mouser part no. 603-CFR-25JT-52-1M -> 603-CFR-25JT-52-1M; Part no. (none) -> CFR-25JT-52-1M
- R12, R2, R3, R5: Mouser part no. 603-MFR-12FTF52-27K -> 603-MFR-12FTF52-27K; Part no. (none) -> MFR-12FTF52-27K
- R13: Mouser part no. 603-RE0805FRE0727KL -> 603-RE0805FRE0727KL; Part no. (none) -> RE0805FRE0727KL
- R4: Mouser part no. 603-MFR-12FTF52-3K6 -> 603-MFR-12FTF52-3K6; Part no. (none) -> MFR-12FTF52-3K6
- R6: Mouser part no. 603-MFR-12FTF52-7K5 -> 603-MFR-12FTF52-7K5; Part no. (none) -> MFR-12FTF52-7K5
- R9: Mouser part no. 603-MFR-12FTF52-56R -> 603-MFR-12FTF52-56R; Part no. (none) -> MFR-12FTF52-56R
- U3: Mouser part no. 595-TL494CPWR -> 595-TL494CPWR; Part no. (none) -> TL494CPWR
Changed lines of the file:
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@@
 			)
 		)
-		(property "Mouser part no." " 637-BC557CBK"
+		(property "Mouser part no." "637-BC557CBK"
+			(at 205.74 92.71 0)
+			(effects
+				(font
+					(size 1.27 1.27)
+				)
+				(hide yes)
+			)
+		)
+		(property "Part no." "BC557CBK"
 			(at 205.74 92.71 0)
 			(effects
@@
 			)
 		)
-		(property "Mouser part no." " 603-MFR-12FTF52-27K"
+		(property "Mouser part no." "603-MFR-12FTF52-27K"
+			(at 118.11 97.79 0)
+			(effects
+				(font
+					(size 1.27 1.27)
+				)
+				(hide yes)
+			)
+		)
+		(property "Part no." "MFR-12FTF52-27K"
 			(at 118.11 97.79 0)
 			(effects
@@
 			)
 		)
-		(property "Mouser part no." " 187-CL21A106KOQNNNE"
+		(property "Mouser part no." "187-CL21A106KOQNNNE"
+			(at 85.09 83.82 0)
+			(effects
+				(font
+					(size 1.27 1.27)
+				)
+				(hide yes)
+			)
+		)
+		(property "Part no." "CL21A106KOQNNNE"
 			(at 85.09 83.82 0)
 			(effects
@@
 			)
 		)
-		(property "Mouser part no." " 710-885012206095"
+		(property "Mouser part no." "710-885012206095"
+			(at 134.62 96.52 0)
+			(effects
+				(font
+					(size 1.27 1.27)
+				)
+				(hide yes)
+			)
+		)
+		(property "Part no." "885012206095"
 			(at 134.62 96.52 0)
 			(effects
@@
 			)
 		)
-		(property "Mouser part no." " 80-C0805C102J5G"
+		(property "Mouser part no." "80-C0805C102J5G"
+			(at 153.67 119.38 0)
+			(effects
+				(font
+					(size 1.27 1.27)
+				)
+				(hide yes)
+			)
+		)
+		(property "Part no." "C0805C102J5G"
 			(at 153.67 119.38 0)
 			(effects
@@
 			)
 		)
-		(property "Mouser part no." " 603-MFR-12FTF52-3K6 "
+		(property "Mouser part no." "603-MFR-12FTF52-3K6"
+			(at 144.78 104.14 0)
+			(effects
+				(font
+					(size 1.27 1.27)
+				)
+				(hide yes)
+			)
+		)
+		(property "Part no." "MFR-12FTF52-3K6"
 			(at 144.78 104.14 0)
 			(effects
@@
 			)
 		)
-		(property "Mouser part no." " 603-MFR-12FTF52-27K"
+		(property "Mouser part no." "603-MFR-12FTF52-27K"
+			(at 187.96 102.87 0)
+			(effects
+				(font
+					(size 1.27 1.27)
+				)
+				(hide yes)
+			)
+		)
+		(property "Part no." "MFR-12FTF52-27K"
 			(at 187.96 102.87 0)
 			(effects
@@
 			)
 		)
-		(property "Mouser part no." " 603-MFR-12FTF52-56R"
+		(property "Mouser part no." "603-MFR-12FTF52-56R"
+			(at 102.87 93.98 0)
+			(effects
+				(font
+					(size 1.27 1.27)
+				)
+				(hide yes)
+			)
+		)
+		(property "Part no." "MFR-12FTF52-56R"
 			(at 102.87 93.98 0)
 			(effects
@@
 			)
 		)
-		(property "Mouser part no." " 603-MFR-12FTF52-27K"
+		(property "Mouser part no." "603-MFR-12FTF52-27K"
+			(at 151.13 85.09 0)
+			(effects
+				(font
+					(size 1.27 1.27)
+				)
+				(hide yes)
+			)
+		)
+		(property "Part no." "MFR-12FTF52-27K"
 			(at 151.13 85.09 0)
 			(effects
@@
 			)
 		)
-		(property "Mouser part no." " 603-MFR-12FTF52-27K"
+		(property "Mouser part no." "603-MFR-12FTF52-27K"
+			(at 194.31 92.71 0)
+			(effects
+				(font
+					(size 1.27 1.27)
+				)
+				(hide yes)
+			)
+		)
+		(property "Part no." "MFR-12FTF52-27K"
 			(at 194.31 92.71 0)
 			(effects
@@
 			)
 		)
-		(property "Mouser part no." " 603-MFR-12FTF52-0R1"
+		(property "Mouser part no." "603-MFR-12FTF52-0R1"
+			(at 91.44 101.6 0)
+			(effects
+				(font
+					(size 1.27 1.27)
+				)
+				(hide yes)
+			)
+		)
+		(property "Part no." "MFR-12FTF52-0R1"
 			(at 91.44 101.6 0)
 			(effects
@@
 			)
 		)
-		(property "Mouser part no." " 603-CFR-25JT-52-1M"
+		(property "Mouser part no." "603-CFR-25JT-52-1M"
+			(at 125.73 96.52 0)
+			(effects
+				(font
+					(size 1.27 1.27)
+				)
+				(hide yes)
+			)
+		)
+		(property "Part no." "CFR-25JT-52-1M"
 			(at 125.73 96.52 0)
 			(effects
@@
 			)
 		)
-		(property "Mouser part no." " 603-RE0805FRE0727KL"
+		(property "Mouser part no." "603-RE0805FRE0727KL"
+			(at 107.95 99.06 0)
+			(effects
+				(font
+					(size 1.27 1.27)
+				)
+				(hide yes)
+			)
+		)
+		(property "Part no." "RE0805FRE0727KL"
 			(at 107.95 99.06 0)
 			(effects
@@
 			)
 		)
-		(property "Mouser part no." " 603-MFR-12FTF52-7K5"
+		(property "Mouser part no." "603-MFR-12FTF52-7K5"
+			(at 118.11 109.22 0)
+			(effects
+				(font
+					(size 1.27 1.27)
+				)
+				(hide yes)
+			)
+		)
+		(property "Part no." "MFR-12FTF52-7K5"
 			(at 118.11 109.22 0)
 			(effects
@@
 			)
 		)
-		(property "Mouser part no." " 603-MFR-12FTF52-12K"
+		(property "Mouser part no." "603-MFR-12FTF52-12K"
+			(at 143.51 119.38 0)
+			(effects
+				(font
+					(size 1.27 1.27)
+				)
+				(hide yes)
+			)
+		)
+		(property "Part no." "MFR-12FTF52-12K"
 			(at 143.51 119.38 0)
 			(effects
@@
 			)
 		)
-		(property "Mouser part no." " 637-BC547CBK"
+		(property "Mouser part no." "637-BC547CBK"
+			(at 205.74 107.95 0)
+			(effects
+				(font
+					(size 1.27 1.27)
+				)
+				(hide yes)
+			)
+		)
+		(property "Part no." "BC547CBK"
 			(at 205.74 107.95 0)
 			(effects
@@
 			)
 		)
-		(property "Mouser part no." " 595-TL494CPWR"
+		(property "Mouser part no." "595-TL494CPWR"
 			(at 167.64 104.14 0)
 			(effects
+				(font
+					(size 1.27 1.27)
+				)
+				(hide yes)
+			)
+		)
+		(property "Part no." "TL494CPWR"
+			(at 167.64 104.14 0)
+			(effects

Commit message: fix BOM, add more LCSC part numbers
Parts:
- C1: LCSC part no. (none) -> C1713
- C3: LCSC part no. (none) -> C599833
- C4: LCSC part no. (none) -> C14663
- Q1: LCSC part no. (none) -> C5595521
- Q2: LCSC part no. (none) -> C3201550
- R1: LCSC part no. (none) -> C1389771
- R10: LCSC part no. (none) -> C2896932
- R11: LCSC part no. (none) -> C714052
- R12, R2, R3, R5: LCSC part no. (none) -> C2896992
- R13: LCSC part no. (none) -> C375523
- R4: LCSC part no. (none) -> C367441
- R6: LCSC part no. (none) -> C714231
- R9: LCSC part no. (none) -> C713895
- U3: LCSC part no. (none) -> C163520
Changed lines of the file:
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@@
+			)
+		)
+		(property "LCSC part no." "C5595521"
+			(at 205.74 92.71 0)
+			(effects
+				(font
+					(size 1.27 1.27)
+				)
+				(hide yes)
 			)
 		)
@@
 			)
 		)
+		(property "LCSC part no." "C2896992"
+			(at 118.11 97.79 0)
+			(effects
+				(font
+					(size 1.27 1.27)
+				)
+				(hide yes)
+			)
+		)
 		(pin "2"
 		)
@@
 			)
 		)
+		(property "LCSC part no." "C1713"
+			(at 85.09 83.82 0)
+			(effects
+				(font
+					(size 1.27 1.27)
+				)
+				(hide yes)
+			)
+		)
 		(pin "2"
 		)
@@
 			)
 		)
+		(property "LCSC part no." "C14663"
+			(at 134.62 96.52 0)
+			(effects
+				(font
+					(size 1.27 1.27)
+				)
+				(hide yes)
+			)
+		)
 		(pin "1"
 		)
@@
 			)
 		)
+		(property "LCSC part no." "C599833"
+			(at 153.67 119.38 0)
+			(effects
+				(font
+					(size 1.27 1.27)
+				)
+				(hide yes)
+			)
+		)
 		(pin "1"
 		)
@@
 			)
 		)
+		(property "LCSC part no." "C367441"
+			(at 144.78 104.14 0)
+			(effects
+				(font
+					(size 1.27 1.27)
+				)
+				(hide yes)
+			)
+		)
 		(pin "2"
 		)
@@
 			)
 		)
+		(property "LCSC part no." "C2896992"
+			(at 187.96 102.87 0)
+			(effects
+				(font
+					(size 1.27 1.27)
+				)
+				(hide yes)
+			)
+		)
 		(pin "2"
 		)
@@
 			)
 		)
+		(property "LCSC part no." "C713895"
+			(at 102.87 93.98 0)
+			(effects
+				(font
+					(size 1.27 1.27)
+				)
+				(hide yes)
+			)
+		)
 		(pin "2"
 		)
@@
 			)
 		)
+		(property "LCSC part no." "C2896992"
+			(at 151.13 85.09 0)
+			(effects
+				(font
+					(size 1.27 1.27)
+				)
+				(hide yes)
+			)
+		)
 		(pin "2"
 		)
@@
 			)
 		)
+		(property "LCSC part no." "C2896992"
+			(at 194.31 92.71 0)
+			(effects
+				(font
+					(size 1.27 1.27)
+				)
+				(hide yes)
+			)
+		)
 		(pin "2"
 		)
@@
 			)
 		)
+		(property "LCSC part no." "C1389771"
+			(at 91.44 101.6 0)
+			(effects
+				(font
+					(size 1.27 1.27)
+				)
+				(hide yes)
+			)
+		)
 		(pin "1"
 		)
@@
 			)
 		)
+		(property "LCSC part no." "C714052"
+			(at 125.73 96.52 0)
+			(effects
+				(font
+					(size 1.27 1.27)
+				)
+				(hide yes)
+			)
+		)
 		(pin "2"
 		)
@@
 			)
 		)
+		(property "LCSC part no." "C375523"
+			(at 107.95 99.06 0)
+			(effects
+				(font
+					(size 1.27 1.27)
+				)
+				(hide yes)
+			)
+		)
 		(pin "2"
 		)
@@
 			)
 		)
+		(property "LCSC part no." "C714231"
+			(at 118.11 109.22 0)
+			(effects
+				(font
+					(size 1.27 1.27)
+				)
+				(hide yes)
+			)
+		)
 		(pin "2"
 		)
@@
 			)
 		)
+		(property "LCSC part no." "C2896932"
+			(at 143.51 119.38 0)
+			(effects
+				(font
+					(size 1.27 1.27)
+				)
+				(hide yes)
+			)
+		)
 		(pin "2"
 		)
@@
 			)
 		)
+		(property "LCSC part no." "C3201550"
+			(at 205.74 107.95 0)
+			(effects
+				(font
+					(size 1.27 1.27)
+				)
+				(hide yes)
+			)
+		)
 		(pin "3"
 		)
@@
 			(at 167.64 104.14 0)
 			(effects
+				(font
+					(size 1.27 1.27)
+				)
+				(hide yes)
+			)
+		)
+		(property "LCSC part no." "C163520"
+			(at 167.64 104.14 0)
+			(effects

Commit message: final? version
Parts:
- added R20: 27k, Resistor_THT:R_Axial_DIN0204_L3.6mm_D1.6mm_P7.62mm_Horizontal, symbol Device:R
Connections:
- net +12V: now also R20.1
- net at R2.1, U3.8 (C1): now also R20.2
Changed lines of the file:
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@@
+	)
+	(junction
+		(at 184.15 92.71)
+		(diameter 0)
+		(color 0 0 0 0)
 	)
 	(junction
@@
 	)
 	(junction
+		(at 184.15 74.93)
+		(diameter 0)
+		(color 0 0 0 0)
+	)
+	(junction
 		(at 107.95 93.98)
 		(diameter 0)
@@
 	(wire
 		(pts
+			(xy 184.15 74.93) (xy 167.64 74.93)
+		)
+		(stroke
+			(width 0)
+			(type default)
+		)
+	)
+	(wire
+		(pts
 			(xy 85.09 72.39) (xy 85.09 74.93)
 		)
@@
 	(wire
 		(pts
+			(xy 184.15 90.17) (xy 184.15 92.71)
+		)
+		(stroke
+			(width 0)
+			(type default)
+		)
+	)
+	(wire
+		(pts
 			(xy 184.15 92.71) (xy 190.5 92.71)
 		)
@@
 	(wire
 		(pts
-			(xy 187.96 74.93) (xy 167.64 74.93)
+			(xy 187.96 74.93) (xy 184.15 74.93)
 		)
 		(stroke
@@
 		(pts
 			(xy 184.15 99.06) (xy 184.15 92.71)
+		)
+		(stroke
+			(width 0)
+			(type default)
+		)
+	)
+	(wire
+		(pts
+			(xy 184.15 74.93) (xy 184.15 82.55)
 		)
 		(stroke
@@
 	)
 	(symbol
+		(lib_id "Device:R")
+		(at 184.15 86.36 0)
+		(unit 1)
+		(exclude_from_sim no)
+		(in_bom yes)
+		(on_board yes)
+		(dnp no)
+		(fields_autoplaced yes)
+		(property "Reference" "R20"
+			(at 186.69 85.0899 0)
+			(effects
+				(font
+					(size 1.27 1.27)
+				)
+				(justify left)
+			)
+		)
+		(property "Value" "27k"
+			(at 186.69 87.6299 0)
+			(effects
+				(font
+					(size 1.27 1.27)
+				)
+				(justify left)
+			)
+		)
+		(property "Footprint" "Resistor_THT:R_Axial_DIN0204_L3.6mm_D1.6mm_P7.62mm_Horizontal"
+			(at 182.372 86.36 90)
+			(effects
+				(font
+					(size 1.27 1.27)
+				)
+				(hide yes)
+			)
+		)
+		(property "Datasheet" "~"
+			(at 184.15 86.36 0)
+			(effects
+				(font
+					(size 1.27 1.27)
+				)
+				(hide yes)
+			)
+		)
+		(property "Description" "Resistor"
+			(at 184.15 86.36 0)
+			(effects
+				(font
+					(size 1.27 1.27)
+				)
+				(hide yes)
+			)
+		)
+		(property "Mouser part no." "603-MFR-12FTF52-27K"
+			(at 184.15 86.36 0)
+			(effects
+				(font
+					(size 1.27 1.27)
+				)
+				(hide yes)
+			)
+		)
+		(property "Part no." "MFR-12FTF52-27K"
+			(at 184.15 86.36 0)
+			(effects
+				(font
+					(size 1.27 1.27)
+				)
+				(hide yes)
+			)
+		)
+		(property "LCSC part no." "C2896992"
+			(at 184.15 86.36 0)
+			(effects
+				(font
+					(size 1.27 1.27)
+				)
+				(hide yes)
+			)
+		)
+		(pin "2"
+		)
+		(pin "1"
+		)
+		(instances
+			(project "osborne-floppy-emulator"
+				(path "/a407fcbc-6d86-4aa2-968f-b2fcdecb9640/ff2c5a00-867d-47b1-bade-a270f3659bc6"
+					(reference "R20")
+					(unit 1)
+				)
+			)
+		)
+	)
+	(symbol
 		(lib_id "power:GND")
 		(at 139.7 120.65 0)
@@
 	)
 	(symbol
+		(lib_name "R_1")
 		(lib_id "Device:R")
 		(at 194.31 92.71 90)
