File: board/sepic2.kicad_sch (KiCad schematic)
At the start: 8 parts, among them Q1 T2N7002BK

Commit message: fix BOM, add column for mfr. part number
Parts:
- C1: Mouser part no. 710-885012206095 -> 710-885012206095; Part no. (none) -> 885012206095
- Cin1: Mouser part no. 710-860080473006 -> 710-860080473006; Part no. (none) -> 860080473006
- Cout1, Cout2: Mouser part no. 187-CL21A106KOQNNNE -> 187-CL21A106KOQNNNE; Part no. (none) -> CL21A106KOQNNNE
- D1: Mouser part no. 833-1N5819-TP -> 833-1N5819-TP; Part no. (none) -> 1N5819-TP
- L1: Mouser part no. 580-50105C -> 580-50105C; Part no. (none) -> 50105C
- L3: Mouser part no. 963-LBR2518T100K -> 963-LBR2518T100K; Part no. (none) -> LBR2518T100K
- Q1: Mouser part no. 757-T2N7002BKLM -> 757-T2N7002BKLM; Part no. (none) -> T2N7002BKLM
Changed lines of the file:
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@@
 			)
 		)
-		(property "Mouser part no." " 580-50105C"
+		(property "Mouser part no." "580-50105C"
+			(at 114.3 48.26 0)
+			(effects
+				(font
+					(size 1.27 1.27)
+				)
+				(hide yes)
+			)
+		)
+		(property "Part no." "50105C"
 			(at 114.3 48.26 0)
 			(effects
@@
 			)
 		)
-		(property "Mouser part no." " 833-1N5819-TP"
+		(property "Mouser part no." "833-1N5819-TP"
+			(at 148.59 41.91 0)
+			(effects
+				(font
+					(size 1.27 1.27)
+				)
+				(hide yes)
+			)
+		)
+		(property "Part no." "1N5819-TP"
 			(at 148.59 41.91 0)
 			(effects
@@
 			)
 		)
-		(property "Mouser part no." " 187-CL21A106KOQNNNE"
+		(property "Mouser part no." "187-CL21A106KOQNNNE"
+			(at 170.18 76.2 0)
+			(effects
+				(font
+					(size 1.27 1.27)
+				)
+				(hide yes)
+			)
+		)
+		(property "Part no." "CL21A106KOQNNNE"
 			(at 170.18 76.2 0)
 			(effects
@@
 			)
 		)
-		(property "Mouser part no." " 187-CL21A106KOQNNNE"
+		(property "Mouser part no." "187-CL21A106KOQNNNE"
+			(at 154.94 76.2 0)
+			(effects
+				(font
+					(size 1.27 1.27)
+				)
+				(hide yes)
+			)
+		)
+		(property "Part no." "CL21A106KOQNNNE"
 			(at 154.94 76.2 0)
 			(effects
@@
 			)
 		)
-		(property "Mouser part no." " 757-T2N7002BKLM"
+		(property "Mouser part no." "757-T2N7002BKLM"
+			(at 106.68 69.85 0)
+			(effects
+				(font
+					(size 1.27 1.27)
+				)
+				(hide yes)
+			)
+		)
+		(property "Part no." "T2N7002BKLM"
 			(at 106.68 69.85 0)
 			(effects
@@
 			)
 		)
-		(property "Mouser part no." " 710-860080473006"
+		(property "Mouser part no." "710-860080473006"
+			(at 71.12 76.2 0)
+			(effects
+				(font
+					(size 1.27 1.27)
+				)
+				(hide yes)
+			)
+		)
+		(property "Part no." "860080473006"
 			(at 71.12 76.2 0)
 			(effects
@@
 			)
 		)
-		(property "Mouser part no." " 963-LBR2518T100K"
+		(property "Mouser part no." "963-LBR2518T100K"
+			(at 162.56 41.91 0)
+			(effects
+				(font
+					(size 1.27 1.27)
+				)
+				(hide yes)
+			)
+		)
+		(property "Part no." "LBR2518T100K"
 			(at 162.56 41.91 0)
 			(effects
@@
 			)
 		)
-		(property "Mouser part no." " 710-885012206095"
+		(property "Mouser part no." "710-885012206095"
 			(at 114.3 57.15 0)
 			(effects
+				(font
+					(size 1.27 1.27)
+				)
+				(hide yes)
+			)
+		)
+		(property "Part no." "885012206095"
+			(at 114.3 57.15 0)
+			(effects

Commit message: fix BOM, add more LCSC part numbers
Parts:
- C1: LCSC part no. (none) -> C14663
- Cin1: LCSC part no. (none) -> C88754
- Cout1, Cout2: LCSC part no. (none) -> C1713
- D1: LCSC part no. (none) -> C526214
- L1: LCSC part no. (none) -> C6393640
- L3: LCSC part no. (none) -> C2041481
- Q1: LCSC part no. (none) -> C146372
Changed lines of the file:
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@@
+			)
+		)
+		(property "LCSC part no." "C6393640"
+			(at 114.3 48.26 0)
+			(effects
+				(font
+					(size 1.27 1.27)
+				)
+				(hide yes)
 			)
 		)
@@
 			)
 		)
+		(property "LCSC part no." "C526214"
+			(at 148.59 41.91 0)
+			(effects
+				(font
+					(size 1.27 1.27)
+				)
+				(hide yes)
+			)
+		)
 		(pin "2"
 		)
@@
 			)
 		)
+		(property "LCSC part no." "C1713"
+			(at 170.18 76.2 0)
+			(effects
+				(font
+					(size 1.27 1.27)
+				)
+				(hide yes)
+			)
+		)
 		(pin "1"
 		)
@@
 			)
 		)
+		(property "LCSC part no." "C1713"
+			(at 154.94 76.2 0)
+			(effects
+				(font
+					(size 1.27 1.27)
+				)
+				(hide yes)
+			)
+		)
 		(pin "1"
 		)
@@
 			)
 		)
+		(property "LCSC part no." "C146372"
+			(at 106.68 69.85 0)
+			(effects
+				(font
+					(size 1.27 1.27)
+				)
+				(hide yes)
+			)
+		)
 		(pin "2"
 		)
@@
 			)
 		)
+		(property "LCSC part no." "C88754"
+			(at 71.12 76.2 0)
+			(effects
+				(font
+					(size 1.27 1.27)
+				)
+				(hide yes)
+			)
+		)
 		(pin "1"
 		)
@@
 		)
 		(property "Part no." "LBR2518T100K"
+			(at 162.56 41.91 0)
+			(effects
+				(font
+					(size 1.27 1.27)
+				)
+				(hide yes)
+			)
+		)
+		(property "LCSC part no." "C2041481"
 			(at 162.56 41.91 0)
 			(effects
@@
 			(at 114.3 57.15 0)
 			(effects
+				(font
+					(size 1.27 1.27)
+				)
+				(hide yes)
+			)
+		)
+		(property "LCSC part no." "C14663"
+			(at 114.3 57.15 0)
+			(effects

Commit message: final? version
Changed lines of the file:
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@@
 		(on_board yes)
 		(dnp no)
+		(fields_autoplaced yes)
 		(property "Reference" "L1"
-			(at 106.68 48.006 0)
-			(effects
-				(font
-					(size 1.27 1.27)
-				)
+			(at 118.11 46.6089 90)
+			(effects
+				(font
+					(size 1.27 1.27)
+				)
+				(justify right)
 			)
 		)
 		(property "Value" "1m"
-			(at 109.22 48.006 0)
-			(effects
-				(font
-					(size 1.27 1.27)
-				)
+			(at 118.11 49.1489 90)
+			(effects
+				(font
+					(size 1.27 1.27)
+				)
+				(justify right)
 			)
 		)
@@
 		(fields_autoplaced yes)
 		(property "Reference" "C1"
-			(at 114.3 49.53 90)
+			(at 114.3 62.23 90)
 			(effects
 				(font
@@
 		)
 		(property "Value" "100n"
-			(at 114.3 52.07 90)
-			(effects
-				(font
+			(at 114.3 64.77 90)
+			(effects
+				(font
